File: hardware/bmp180.sch (KiCad schematic (older format))
At the start: 0 parts

Commit message: update,
Parts:
- added C?: C104,0603, Capacitor_SMD:C_0603_1608Metric_Pad1.05x0.95mm_HandSolder, symbol taobao-c:C104,0603
- added J?: BMP180_HEADER, Connector_PinHeader_1.27mm:PinHeader_1x04_P1.27mm_Vertical, symbol Connector:Conn_01x04_Female
- added RN?: RN_103,0603, Resistor_SMD:R_Array_Concave_4x0603, symbol taobao-rpack:RN_103,0603
- added U?: BMP180, footprint-lib:BMP180, symbol taobao-components:BMP180
Connections:
- new net +3V3: C?.2, J?.1 (Pin_1), RN?.7 (R2.2), RN?.8 (R1.2), U?.2 (VDD), U?.3 (VDDIO)
- new net GND: C?.1, J?.2 (Pin_2), U?.7 (GND)
- new net SCL: J?.3 (Pin_3), RN?.1 (R1.1), U?.5 (SCL)
- new net SDA: J?.4 (Pin_4), RN?.2 (R2.1), U?.6 (SDA)
- no-connect marks 0 -> 6
