File: hardware/bmp180.sch (KiCad schematic (older format))
At the start: 4 parts

Commit message: update,
Parts:
- gave numbers to parts that had none: 4
Changed lines of the file:
@@
 EESchema Schematic File Version 4
-LIBS:PMS5003S_MOUNT-cache
-LIBS:bmp180_tryout-cache
+LIBS:cowin-tryout-cache
+LIBS:CH340T-tryout-cache
 EELAYER 29 0
 EELAYER END
 $Descr User 8500 5500
 encoding utf-8
-Sheet 2 8
+Sheet 2 12
 Title ""
 Date ""
@@
 $EndBitmap
 $Comp
-L taobao-components:BMP180 U?
+L taobao-components:BMP180 U1
 U 1 1 5D137C1E
 P 3050 2000
-F 0 "U?" H 3050 2715 50  0000 C CNN
+F 0 "U1" H 3050 2715 50  0000 C CNN
 F 1 "BMP180" H 3050 2624 50  0000 C CNN
 F 2 "footprint-lib:BMP180" H 3050 1350 50  0001 C CNN
@@
 $EndComp
 $Comp
-L taobao-rpack:RN_103,0603 RN?
+L taobao-rpack:RN_103,0603 RN1
 U 1 1 5D138380
 P 4400 1550
-F 0 "RN?" H 4588 1596 50  0000 L CNN
+F 0 "RN1" H 4588 1596 50  0000 L CNN
 F 1 "RN_103,0603" H 4588 1505 50  0000 L CNN
 F 2 "Resistor_SMD:R_Array_Concave_4x0603" V 4675 1550 50  0001 C CNN
@@
 $EndComp
 $Comp
-L power:+3V3 #PWR?
+L power:+3V3 #PWR0101
 U 1 1 5D1392D6
 P 3900 1000
-F 0 "#PWR?" H 3900 850 50  0001 C CNN
+F 0 "#PWR0101" H 3900 850 50  0001 C CNN
 F 1 "+3V3" H 3915 1173 50  0000 C CNN
 F 2 "" H 3900 1000 50  0001 C CNN
@@
 $EndComp
 $Comp
-L power:GND #PWR?
+L power:GND #PWR0102
 U 1 1 5D13998C
 P 3850 2450
-F 0 "#PWR?" H 3850 2200 50  0001 C CNN
+F 0 "#PWR0102" H 3850 2200 50  0001 C CNN
 F 1 "GND" H 3855 2277 50  0000 C CNN
 F 2 "" H 3850 2450 50  0001 C CNN
@@
 $EndComp
 $Comp
-L Connector:Conn_01x04_Female J?
+L Connector:Conn_01x04_Female J1
 U 1 1 5D139F4B
 P 1400 1900
-F 0 "J?" H 1292 2185 50  0000 C CNN
+F 0 "J1" H 1292 2185 50  0000 C CNN
 F 1 "BMP180_HEADER" H 1292 2094 50  0000 C CNN
 F 2 "Connector_PinHeader_1.27mm:PinHeader_1x04_P1.27mm_Vertical" H 1400 1900 50  0001 C CNN
@@
 $EndComp
 $Comp
-L power:+3V3 #PWR?
+L power:+3V3 #PWR0103
 U 1 1 5D13A64B
 P 1800 1650
-F 0 "#PWR?" H 1800 1500 50  0001 C CNN
+F 0 "#PWR0103" H 1800 1500 50  0001 C CNN
 F 1 "+3V3" H 1815 1823 50  0000 C CNN
 F 2 "" H 1800 1650 50  0001 C CNN
@@
 $EndComp
 $Comp
-L power:GND #PWR?
+L power:GND #PWR0104
 U 1 1 5D13A995
 P 2000 1900
-F 0 "#PWR?" H 2000 1650 50  0001 C CNN
+F 0 "#PWR0104" H 2000 1650 50  0001 C CNN
 F 1 "GND" V 2005 1772 50  0000 R CNN
 F 2 "" H 2000 1900 50  0001 C CNN
@@
 	3900 1650 3900 1200
 $Comp
-L power:+3V3 #PWR?
+L power:+3V3 #PWR0105
 U 1 1 5D13D2C2
 P 2800 1150
-F 0 "#PWR?" H 2800 1000 50  0001 C CNN
+F 0 "#PWR0105" H 2800 1000 50  0001 C CNN
 F 1 "+3V3" V 2815 1278 50  0000 L CNN
 F 2 "" H 2800 1150 50  0001 C CNN
@@
 $EndComp
 $Comp
-L taobao-c:C104,0603 C?
+L taobao-c:C104,0603 C1
 U 1 1 5D13D83D
 P 3000 1150
-F 0 "C?" V 2771 1150 50  0000 C CNN
+F 0 "C1" V 2771 1150 50  0000 C CNN
 F 1 "C104,0603" V 2862 1150 50  0000 C CNN
 F 2 "Capacitor_SMD:C_0603_1608Metric_Pad1.05x0.95mm_HandSolder" H 3000 1150 50  0001 C CNN
@@
 $EndComp
 $Comp
-L power:GND #PWR?
+L power:GND #PWR0106
 U 1 1 5D13DCCD
 P 3250 1150
-F 0 "#PWR?" H 3250 900 50  0001 C CNN
+F 0 "#PWR0106" H 3250 900 50  0001 C CNN
 F 1 "GND" V 3255 1022 50  0000 R CNN
 F 2 "" H 3250 1150 50  0001 C CNN

Commit message: update,
Connections:
- net SCL: now also RN1.2 (R2.1); no longer RN1.1 (R1.1)
- net SDA: now also RN1.1 (R1.1); no longer RN1.2 (R2.1)
Other:
- moved on the sheet: RN1
Changed lines of the file:
@@
 L taobao-rpack:RN_103,0603 RN1
 U 1 1 5D138380
-P 4400 1550
-F 0 "RN1" H 4588 1596 50  0000 L CNN
-F 1 "RN_103,0603" H 4588 1505 50  0000 L CNN
-F 2 "Resistor_SMD:R_Array_Concave_4x0603" V 4675 1550 50  0001 C CNN
-F 3 "~" H 4400 1550 50  0001 C CNN
-	1    4400 1550
-	1    0    0    -1
+P 4100 1550
+F 0 "RN1" H 4288 1596 50  0000 L CNN
+F 1 "RN_103,0603" H 4288 1505 50  0000 L CNN
+F 2 "Resistor_SMD:R_Array_Concave_4x0603" V 4375 1550 50  0001 C CNN
+F 3 "~" H 4100 1550 50  0001 C CNN
+	1    4100 1550
+	-1   0    0    -1
 $EndComp
 $Comp
@@
 Wire Wire Line
 	3550 2150 4300 2150
-NoConn ~ 4400 1350
-NoConn ~ 4500 1350
-NoConn ~ 4400 1750
-NoConn ~ 4500 1750
+NoConn ~ 4100 1350
+NoConn ~ 4000 1350
+NoConn ~ 4100 1750
+NoConn ~ 4000 1750
 NoConn ~ 2550 1550
 NoConn ~ 2550 1850

Commit message: update,
Connections:
- net +3V3: now also RN1.5 (R4.2), RN1.6 (R3.2)
- no-connect marks 6 -> 4
Changed lines of the file:
@@
 Connection ~ 3900 1650
 Wire Wire Line
-	3900 1200 4200 1200
+	3900 1200 4000 1200
 Wire Wire Line
 	4300 1200 4300 1350
@@
 Wire Wire Line
 	3550 2150 4300 2150
-NoConn ~ 4100 1350
-NoConn ~ 4000 1350
 NoConn ~ 4100 1750
 NoConn ~ 4000 1750
@@
 	4600 2150 4300 2150
 Connection ~ 4300 2150
+Wire Wire Line
+	4100 1350 4100 1200
+Connection ~ 4100 1200
+Wire Wire Line
+	4100 1200 4200 1200
+Wire Wire Line
+	4000 1350 4000 1200
+Connection ~ 4000 1200
+Wire Wire Line
+	4000 1200 4100 1200
 $EndSCHEMATC
