File: hardware/cowin-tryout.sch (KiCad schematic (older format))
At the start: 0 parts

Commit message: update,
Changed lines of the file:
@@
 EESchema Schematic File Version 4
 LIBS:PMS5003S_MOUNT-cache
+LIBS:bmp180_tryout-cache
 EELAYER 29 0
 EELAYER END
 $Descr A4 11693 8268
 encoding utf-8
-Sheet 1 5
+Sheet 1 6
 Title ""
 Date ""
@@
 $EndDescr
 $Sheet
-S 8350 1200 850  650
-U 5D1442C0
-F0 "sht3x" 50
-F1 "sht3x.sch" 50
-$EndSheet
-$Sheet
 S 8350 2200 850  650
 U 5D1442CD
 F0 "bmp180" 50
 F1 "bmp180.sch" 50
+F2 "SCL" I L 8350 2450 50
+F3 "SDA" I L 8350 2550 50
 $EndSheet
 $Sheet
@@
 F0 "sunlight_uv" 50
 F1 "sunlight_uv.sch" 50
+F2 "ADC" I L 8350 3500 50
+F3 "EN" I L 8350 3600 50
 $EndSheet
 $Sheet
@@
 F0 "pm2_5" 50
 F1 "pm2_5.sch" 50
+F2 "SEN_SET" I L 8350 4550 50
+F3 "SEN_RXD" I L 8350 4650 50
+F4 "SEN_TXD" I L 8350 4750 50
+F5 "SEN_RESET" I L 8350 4850 50
+$EndSheet
+$Sheet
+S 8350 1300 850  650
+U 5D1735E0
+F0 "SHT3X" 50
+F1 "SHT3X.sch" 50
+F2 "SCL" I L 8350 1550 50
+F3 "SDA" I L 8350 1650 50
+$EndSheet
+$Sheet
+S 8350 5350 850  500
+U 5D17F36B
+F0 "terminal" 50
+F1 "terminal.sch" 50
 $EndSheet
 $EndSCHEMATC
