File: hardware/cowin-tryout.sch (KiCad schematic (older format))
At the start: 0 parts

Commit message: update,
Parts:
- added H1, H2, H3, H4: MOUNT_M2.5, footprint-lib:MountingHole_2.7mm_M2.5,rpi_like, symbol taobao-mounting-hole:MOUNT_M2.5
- added U?: DESIGNED_IN_HONG_KONG, symbol taobao-board:DESIGNED_IN_HONG_KONG
- added U?: GITHUB_ADDRESS, symbol taobao-board:GITHUB_ADDRESS
- added U?: BOARD_REVISION, symbol taobao-board:BOARD_REVISION

Commit message: update,
Changed lines of the file:
@@
 EESchema Schematic File Version 4
 LIBS:cowin-tryout-cache
-LIBS:CH340T-tryout-cache
 EELAYER 29 0
 EELAYER END
@@
 $EndSheet
 $Sheet
-S 8350 4000 850  500
+S 8350 4000 750  650
 U 5D17F36B
 F0 "terminal" 50
@@
 F2 "SCL" I L 8350 4150 50
 F3 "SDA" I L 8350 4250 50
+F4 "TXD" I L 8350 4400 50
+F5 "RXD" I L 8350 4500 50
 $EndSheet
 $Sheet
@@
 	1    0    0    -1
 $EndComp
-Wire Bus Line
-	5450 900  5450 2850
-Wire Bus Line
-	7650 900  7650 4450
 $Comp
 L taobao-board:BOARD_REVISION U?
@@
 	1    0    0    -1
 $EndComp
+Entry Wire Line
+	7650 4300 7750 4400
+Entry Wire Line
+	7650 4400 7750 4500
+Wire Wire Line
+	7750 4400 8350 4400
+Wire Wire Line
+	7750 4500 8350 4500
+Text Label 7950 4400 0    50   ~ 0
+TXD
+Text Label 7950 4500 0    50   ~ 0
+RXD
+Wire Bus Line
+	5450 900  5450 2850
+Wire Bus Line
+	7650 900  7650 4700
 $EndSCHEMATC

Commit message: update,
Parts:
- gave numbers to parts that had none: 2
Changed lines of the file:
@@
 $EndSheet
 $Comp
-L taobao-board:DESIGNED_IN_HONG_KONG U?
+L taobao-board:DESIGNED_IN_HONG_KONG U12
 U 1 1 5D1FB661
 P 4050 6800
-F 0 "U?" H 4178 6846 50  0000 L CNN
+F 0 "U12" H 4178 6846 50  0000 L CNN
 F 1 "DESIGNED_IN_HONG_KONG" H 4178 6755 50  0000 L CNN
 F 2 "" H 4050 6650 50  0001 C CNN
@@
 $EndComp
 $Comp
-L taobao-board:GITHUB_ADDRESS U?
+L taobao-board:GITHUB_ADDRESS U13
 U 1 1 5D1FB900
 P 4050 7100
-F 0 "U?" H 4178 7146 50  0000 L CNN
+F 0 "U13" H 4178 7146 50  0000 L CNN
 F 1 "GITHUB_ADDRESS" H 4178 7055 50  0000 L CNN
 F 2 "" H 4050 6900 50  0001 C CNN

Commit message: update,
Parts:
- U12: footprint (none) -> footprint-lib:DESIGNED_IN_HONG_KONG
- U13: footprint (none) -> footprint-lib:GITHUB_ADDRESS
- U15: renamed from U?; footprint (none) -> footprint-lib:BOARD_REVISION
Changed lines of the file:
@@
 EESchema Schematic File Version 4
 LIBS:cowin-tryout-cache
+LIBS:CH340T-tryout-cache
+LIBS:MCP73831-cache
 EELAYER 29 0
 EELAYER END
 $Descr A4 11693 8268
 encoding utf-8
-Sheet 1 12
+Sheet 1 13
 Title ""
 Date ""
@@
 F 0 "U12" H 4178 6846 50  0000 L CNN
 F 1 "DESIGNED_IN_HONG_KONG" H 4178 6755 50  0000 L CNN
-F 2 "" H 4050 6650 50  0001 C CNN
+F 2 "footprint-lib:DESIGNED_IN_HONG_KONG" H 4050 6650 50  0001 C CNN
 F 3 "" H 4050 6650 50  0001 C CNN
 	1    4050 6800
@@
 F 0 "U13" H 4178 7146 50  0000 L CNN
 F 1 "GITHUB_ADDRESS" H 4178 7055 50  0000 L CNN
-F 2 "" H 4050 6900 50  0001 C CNN
+F 2 "footprint-lib:GITHUB_ADDRESS" H 4050 6900 50  0001 C CNN
 F 3 "" H 4050 6900 50  0001 C CNN
 	1    4050 7100
@@
 $EndComp
 $Comp
-L taobao-board:BOARD_REVISION U?
+L taobao-board:BOARD_REVISION U15
 U 1 1 5D1FD10E
 P 4050 7400
-F 0 "U?" H 4178 7446 50  0000 L CNN
+F 0 "U15" H 4178 7446 50  0000 L CNN
 F 1 "BOARD_REVISION" H 4178 7355 50  0000 L CNN
-F 2 "" H 4050 7150 50  0001 C CNN
+F 2 "footprint-lib:BOARD_REVISION" H 4050 7150 50  0001 C CNN
 F 3 "" H 4050 7150 50  0001 C CNN
 	1    4050 7400
@@
 Text Label 7950 4500 0    50   ~ 0
 RXD
+$Sheet
+S 2250 6600 1050 800
+U 5D200348
+F0 "MCP73831" 50
+F1 "MCP73831.sch" 50
+$EndSheet
 Wire Bus Line
 	5450 900  5450 2850

Commit message: update,
Changed lines of the file:
@@
 EESchema Schematic File Version 4
 LIBS:cowin-tryout-cache
-LIBS:CH340T-tryout-cache
-LIBS:MCP73831-cache
 EELAYER 29 0
 EELAYER END
 $Descr A4 11693 8268
 encoding utf-8
-Sheet 1 13
+Sheet 1 14
 Title ""
 Date ""
@@
 F1 "MCP73831.sch" 50
 $EndSheet
+$Sheet
+S 8350 5000 750  650
+U 5D19E051
+F0 "at24cxx" 50
+F1 "at24cxx.sch" 50
+F2 "SCL" I L 8350 5250 50
+F3 "SDA" I L 8350 5350 50
+$EndSheet
+Entry Wire Line
+	7650 5150 7750 5250
+Entry Wire Line
+	7650 5250 7750 5350
+Wire Wire Line
+	7750 5250 8350 5250
+Wire Wire Line
+	7750 5350 8350 5350
+Text Label 7950 5250 0    50   ~ 0
+SCL
+Text Label 7950 5350 0    50   ~ 0
+SDA
 Wire Bus Line
 	5450 900  5450 2850
 Wire Bus Line
-	7650 900  7650 4700
+	7650 900  7650 5350
 $EndSCHEMATC

Commit message: update,
Changed lines of the file:
@@
 $Descr A4 11693 8268
 encoding utf-8
-Sheet 1 14
+Sheet 1 15
 Title ""
 Date ""
@@
 F8 "GPIO14" I L 3300 1600 50
 F9 "GPIO12" I R 4300 2600 50
-F10 "GPIO13" I L 3300 2350 50
+F10 "GPIO13" I R 4300 2200 50
 $EndSheet
 Wire Wire Line
@@
 Text Label 7950 5350 0    50   ~ 0
 SDA
+$Sheet
+S 8350 5900 750  550
+U 5D1B62BF
+F0 "DHT22" 50
+F1 "DHT22.sch" 50
+F2 "DOUT" I L 8350 6150 50
+$EndSheet
+Entry Wire Line
+	7650 6050 7750 6150
+Wire Wire Line
+	7750 6150 8350 6150
+Text Label 7950 6150 0    50   ~ 0
+DHT_OUT
+Entry Wire Line
+	5450 2100 5350 2200
+Wire Wire Line
+	4300 2200 5350 2200
+Text Label 5300 2200 2    50   ~ 0
+DHT_OUT
 Wire Bus Line
 	5450 900  5450 2850
 Wire Bus Line
-	7650 900  7650 5350
+	7650 900  7650 6200
 $EndSCHEMATC
