File: hardware/sunlight_uv.sch (KiCad schematic (older format))
At the start: 0 parts

Commit message: update,
Parts:
- added C?: C104,0603, Capacitor_SMD:C_0603_1608Metric_Pad1.05x0.95mm_HandSolder, symbol taobao-c:C104,0603
- added C?: C102,0603, Capacitor_SMD:C_0603_1608Metric_Pad1.05x0.95mm_HandSolder, symbol taobao-c:C102,0603
- added R?: R103,0603, Resistor_SMD:R_0603_1608Metric_Pad1.05x0.95mm_HandSolder, symbol taobao-r:R103,0603
- added U?: ML8511, footprint-lib:ML8511, symbol taobao-components:ML8511
Connections:
- new net: C?.1, U?.10 (TR)
- new net +3V3: C?.1, R?.1, U?.7 (VDD)
- new net ADC: U?.8 (OUT)
- new net EN: R?.2, U?.4 (EN)
- new net GND: C?.2, C?.2, U?.5 (GND)
- no-connect marks 0 -> 1
