File: hardware/sunlight_uv.sch (KiCad schematic (older format))
At the start: 4 parts

Commit message: update,
Parts:
- gave numbers to parts that had none: 4
Changed lines of the file:
@@
 EESchema Schematic File Version 4
-LIBS:PMS5003S_MOUNT-cache
-LIBS:bmp180_tryout-cache
+LIBS:cowin-tryout-cache
+LIBS:CH340T-tryout-cache
 EELAYER 29 0
 EELAYER END
 $Descr User 8500 5500
 encoding utf-8
-Sheet 3 8
+Sheet 3 12
 Title ""
 Date ""
@@
 $EndBitmap
 $Comp
-L taobao-components:ML8511 U?
+L taobao-components:ML8511 U2
 U 1 1 5D187ABA
 P 4050 2250
-F 0 "U?" H 4025 1511 50  0000 C CNN
+F 0 "U2" H 4025 1511 50  0000 C CNN
 F 1 "ML8511" H 4025 1420 50  0000 C CNN
 F 2 "footprint-lib:ML8511" H 4050 1300 50  0001 C CNN
@@
 $EndComp
 $Comp
-L taobao-c:C104,0603 C?
+L taobao-c:C104,0603 C2
 U 1 1 5D188057
 P 2900 2250
-F 0 "C?" H 2992 2296 50  0000 L CNN
+F 0 "C2" H 2992 2296 50  0000 L CNN
 F 1 "C104,0603" H 2992 2205 50  0000 L CNN
 F 2 "Capacitor_SMD:C_0603_1608Metric_Pad1.05x0.95mm_HandSolder" H 2900 2250 50  0001 C CNN
@@
 $EndComp
 $Comp
-L taobao-c:C102,0603 C?
+L taobao-c:C102,0603 C3
 U 1 1 5D188467
 P 4050 3250
-F 0 "C?" H 4142 3296 50  0000 L CNN
+F 0 "C3" H 4142 3296 50  0000 L CNN
 F 1 "C102,0603" H 4142 3205 50  0000 L CNN
 F 2 "Capacitor_SMD:C_0603_1608Metric_Pad1.05x0.95mm_HandSolder" H 4050 3250 50  0001 C CNN
@@
 $EndComp
 $Comp
-L power:GND #PWR?
+L power:GND #PWR0107
 U 1 1 5D188918
 P 2900 3600
-F 0 "#PWR?" H 2900 3350 50  0001 C CNN
+F 0 "#PWR0107" H 2900 3350 50  0001 C CNN
 F 1 "GND" H 2905 3427 50  0000 C CNN
 F 2 "" H 2900 3600 50  0001 C CNN
@@
 	4700 2500 4950 2500
 $Comp
-L power:+3V3 #PWR?
+L power:+3V3 #PWR0108
 U 1 1 5D18AE40
 P 2900 1700
-F 0 "#PWR?" H 2900 1550 50  0001 C CNN
+F 0 "#PWR0108" H 2900 1550 50  0001 C CNN
 F 1 "+3V3" H 2915 1873 50  0000 C CNN
 F 2 "" H 2900 1700 50  0001 C CNN
@@
 Connection ~ 2900 2000
 $Comp
-L power:+3V3 #PWR?
+L power:+3V3 #PWR0109
 U 1 1 5D18B7BD
 P 4950 1350
-F 0 "#PWR?" H 4950 1200 50  0001 C CNN
+F 0 "#PWR0109" H 4950 1200 50  0001 C CNN
 F 1 "+3V3" H 4965 1523 50  0000 C CNN
 F 2 "" H 4950 1350 50  0001 C CNN
@@
 $EndComp
 $Comp
-L taobao-r:R103,0603 R?
+L taobao-r:R103,0603 R1
 U 1 1 5D18C3A2
 P 4950 1500
-F 0 "R?" H 5009 1546 50  0000 L CNN
+F 0 "R1" H 5009 1546 50  0000 L CNN
 F 1 "R103,0603" H 5009 1455 50  0000 L CNN
 F 2 "Resistor_SMD:R_0603_1608Metric_Pad1.05x0.95mm_HandSolder" H 4950 1500 50  0001 C CNN
