File: hardware/SHT3X.sch (KiCad schematic (older format))
At the start: 6 parts

Commit message: update,
Parts:
- gave numbers to parts that had none: 6
Changed lines of the file:
@@
 EESchema Schematic File Version 4
-LIBS:PMS5003S_MOUNT-cache
-LIBS:bmp180_tryout-cache
+LIBS:cowin-tryout-cache
+LIBS:CH340T-tryout-cache
 EELAYER 29 0
 EELAYER END
 $Descr User 8500 5500
 encoding utf-8
-Sheet 5 8
+Sheet 5 12
 Title ""
 Date ""
@@
 $EndBitmap
 $Comp
-L taobao-components:SHT3x-DIS U?
+L taobao-components:SHT3x-DIS U4
 U 1 1 5CFA0226
 P 3750 2150
-AR Path="/5D1735E0/5CFA0226" Ref="U?"  Part="1"
+AR Path="/5D1735E0/5CFA0226" Ref="U4"  Part="1"
 AR Path="/5D190D23/5CFA0226" Ref="U?"  Part="1"
-F 0 "U?" H 3750 2715 50  0000 C CNN
+F 0 "U4" H 3750 2715 50  0000 C CNN
 F 1 "SHT3x-DIS" H 3750 2624 50  0000 C CNN
 F 2 "footprint-lib:SHT3x-DIS" H 4550 1500 50  0001 C CNN
@@
 $EndComp
 $Comp
-L power:GND #PWR?
+L power:GND #PWR0120
 U 1 1 5CFA0C01
 P 3750 3050
-AR Path="/5D1735E0/5CFA0C01" Ref="#PWR?"  Part="1"
+AR Path="/5D1735E0/5CFA0C01" Ref="#PWR0120"  Part="1"
 AR Path="/5D190D23/5CFA0C01" Ref="#PWR?"  Part="1"
-F 0 "#PWR?" H 3750 2800 50  0001 C CNN
+F 0 "#PWR0120" H 3750 2800 50  0001 C CNN
 F 1 "GND" H 3755 2877 50  0000 C CNN
 F 2 "" H 3750 3050 50  0001 C CNN
@@
 $EndComp
 $Comp
-L power:GND #PWR?
+L power:GND #PWR0121
 U 1 1 5CFA0FDE
 P 2950 3050
-AR Path="/5D1735E0/5CFA0FDE" Ref="#PWR?"  Part="1"
+AR Path="/5D1735E0/5CFA0FDE" Ref="#PWR0121"  Part="1"
 AR Path="/5D190D23/5CFA0FDE" Ref="#PWR?"  Part="1"
-F 0 "#PWR?" H 2950 2800 50  0001 C CNN
+F 0 "#PWR0121" H 2950 2800 50  0001 C CNN
 F 1 "GND" H 2955 2877 50  0000 C CNN
 F 2 "" H 2950 3050 50  0001 C CNN
@@
 $EndComp
 $Comp
-L power:GND #PWR?
+L power:GND #PWR0122
 U 1 1 5CFA11DA
 P 4600 3050
-AR Path="/5D1735E0/5CFA11DA" Ref="#PWR?"  Part="1"
+AR Path="/5D1735E0/5CFA11DA" Ref="#PWR0122"  Part="1"
 AR Path="/5D190D23/5CFA11DA" Ref="#PWR?"  Part="1"
-F 0 "#PWR?" H 4600 2800 50  0001 C CNN
+F 0 "#PWR0122" H 4600 2800 50  0001 C CNN
 F 1 "GND" H 4605 2877 50  0000 C CNN
 F 2 "" H 4600 3050 50  0001 C CNN
@@
 	2950 2450 3100 2450
 $Comp
-L taobao-rpack:RN_472,0603 RN?
+L taobao-rpack:RN_472,0603 RN2
 U 1 1 5CFA1908
 P 2050 1500
-AR Path="/5D1735E0/5CFA1908" Ref="RN?"  Part="1"
+AR Path="/5D1735E0/5CFA1908" Ref="RN2"  Part="1"
 AR Path="/5D190D23/5CFA1908" Ref="RN?"  Part="1"
-F 0 "RN?" H 2238 1546 50  0000 L CNN
+F 0 "RN2" H 2238 1546 50  0000 L CNN
 F 1 "RN_472,0603" H 2238 1455 50  0000 L CNN
 F 2 "Resistor_SMD:R_Array_Concave_4x0603" V 2325 1500 50  0001 C CNN
@@
 	4400 2250 4900 2250
 $Comp
-L power:+3V3 #PWR?
+L power:+3V3 #PWR0123
 U 1 1 5CFA3064
 P 1900 650
-AR Path="/5D1735E0/5CFA3064" Ref="#PWR?"  Part="1"
+AR Path="/5D1735E0/5CFA3064" Ref="#PWR0123"  Part="1"
 AR Path="/5D190D23/5CFA3064" Ref="#PWR?"  Part="1"
-F 0 "#PWR?" H 1900 500 50  0001 C CNN
+F 0 "#PWR0123" H 1900 500 50  0001 C CNN
 F 1 "+3V3" H 1915 823 50  0000 C CNN
 F 2 "" H 1900 650 50  0001 C CNN
@@
 $EndComp
 $Comp
-L my_solder_jumper:SolderJumper_2_Open_round JP?
+L my_solder_jumper:SolderJumper_2_Open_round JP1
 U 1 1 5CFA372A
 P 1900 1000
-AR Path="/5D1735E0/5CFA372A" Ref="JP?"  Part="1"
+AR Path="/5D1735E0/5CFA372A" Ref="JP1"  Part="1"
 AR Path="/5D190D23/5CFA372A" Ref="JP?"  Part="1"
-F 0 "JP?" V 1854 1068 50  0000 L CNN
+F 0 "JP1" V 1854 1068 50  0000 L CNN
 F 1 "SolderJumper_2_Open_round" V 1945 1068 50  0000 L CNN
 F 2 "Jumper:SolderJumper-2_P1.3mm_Open_RoundedPad1.0x1.5mm" H 1900 1000 50  0001 C CNN
@@
 Connection ~ 1900 1200
 $Comp
-L power:+3V3 #PWR?
+L power:+3V3 #PWR0124
 U 1 1 5CFA5513
 P 4600 1600
-AR Path="/5D1735E0/5CFA5513" Ref="#PWR?"  Part="1"
+AR Path="/5D1735E0/5CFA5513" Ref="#PWR0124"  Part="1"
 AR Path="/5D190D23/5CFA5513" Ref="#PWR?"  Part="1"
-F 0 "#PWR?" H 4600 1450 50  0001 C CNN
+F 0 "#PWR0124" H 4600 1450 50  0001 C CNN
 F 1 "+3V3" H 4615 1773 50  0000 C CNN
 F 2 "" H 4600 1600 50  0001 C CNN
@@
 	4600 1850 4600 1600
 $Comp
-L power:+3V3 #PWR?
+L power:+3V3 #PWR0125
 U 1 1 5CFA6101
 P 3450 1350
-AR Path="/5D1735E0/5CFA6101" Ref="#PWR?"  Part="1"
+AR Path="/5D1735E0/5CFA6101" Ref="#PWR0125"  Part="1"
 AR Path="/5D190D23/5CFA6101" Ref="#PWR?"  Part="1"
-F 0 "#PWR?" H 3450 1200 50  0001 C CNN
+F 0 "#PWR0125" H 3450 1200 50  0001 C CNN
 F 1 "+3V3" V 3465 1478 50  0000 L CNN
 F 2 "" H 3450 1350 50  0001 C CNN
@@
 $EndComp
 $Comp
-L power:GND #PWR?
+L power:GND #PWR0126
 U 1 1 5CFA6490
 P 4000 1350
-AR Path="/5D1735E0/5CFA6490" Ref="#PWR?"  Part="1"
+AR Path="/5D1735E0/5CFA6490" Ref="#PWR0126"  Part="1"
 AR Path="/5D190D23/5CFA6490" Ref="#PWR?"  Part="1"
-F 0 "#PWR?" H 4000 1100 50  0001 C CNN
+F 0 "#PWR0126" H 4000 1100 50  0001 C CNN
 F 1 "GND" V 4005 1222 50  0000 R CNN
 F 2 "" H 4000 1350 50  0001 C CNN
@@
 $EndComp
 $Comp
-L taobao-c:C104,0805 C?
+L taobao-c:C104,0805 C5
 U 1 1 5CFA71B1
 P 3700 1350
-AR Path="/5D1735E0/5CFA71B1" Ref="C?"  Part="1"
+AR Path="/5D1735E0/5CFA71B1" Ref="C5"  Part="1"
 AR Path="/5D190D23/5CFA71B1" Ref="C?"  Part="1"
-F 0 "C?" V 3471 1350 50  0000 C CNN
+F 0 "C5" V 3471 1350 50  0000 C CNN
 F 1 "C104,0805" V 3562 1350 50  0000 C CNN
 F 2 "Capacitor_SMD:C_0805_2012Metric_Pad1.15x1.40mm_HandSolder" H 3700 1350 50  0001 C CNN
@@
 ADDR
 $Comp
-L my_solder_jumper:SolderJumper_2_Open_round JP?
+L my_solder_jumper:SolderJumper_2_Open_round JP2
 U 1 1 5CFABF79
 P 2300 2550
-AR Path="/5D1735E0/5CFABF79" Ref="JP?"  Part="1"
+AR Path="/5D1735E0/5CFABF79" Ref="JP2"  Part="1"
 AR Path="/5D190D23/5CFABF79" Ref="JP?"  Part="1"
-F 0 "JP?" V 2254 2618 50  0000 L CNN
+F 0 "JP2" V 2254 2618 50  0000 L CNN
 F 1 "J_ADDR" V 2345 2618 50  0000 L CNN
 F 2 "Jumper:SolderJumper-2_P1.3mm_Open_RoundedPad1.0x1.5mm" H 2300 2550 50  0001 C CNN
@@
 $EndComp
 $Comp
-L power:GND #PWR?
+L power:GND #PWR0127
 U 1 1 5CFAC548
 P 2300 3050
-AR Path="/5D1735E0/5CFAC548" Ref="#PWR?"  Part="1"
+AR Path="/5D1735E0/5CFAC548" Ref="#PWR0127"  Part="1"
 AR Path="/5D190D23/5CFAC548" Ref="#PWR?"  Part="1"
-F 0 "#PWR?" H 2300 2800 50  0001 C CNN
+F 0 "#PWR0127" H 2300 2800 50  0001 C CNN
 F 1 "GND" H 2305 2877 50  0000 C CNN
 F 2 "" H 2300 3050 50  0001 C CNN
@@
 	1950 1700 1950 2050
 $Comp
-L Connector:Conn_01x06_Female J?
+L Connector:Conn_01x06_Female J3
 U 1 1 5CFBB0DE
 P 1250 2750
-AR Path="/5D1735E0/5CFBB0DE" Ref="J?"  Part="1"
+AR Path="/5D1735E0/5CFBB0DE" Ref="J3"  Part="1"
 AR Path="/5D190D23/5CFBB0DE" Ref="J?"  Part="1"
-F 0 "J?" H 1142 3135 50  0000 C CNN
+F 0 "J3" H 1142 3135 50  0000 C CNN
 F 1 "SHT3x_HEADER" H 1142 3044 50  0000 C CNN
 F 2 "Connector_PinHeader_1.27mm:PinHeader_1x06_P1.27mm_Vertical" H 1250 2750 50  0001 C CNN
@@
 $EndComp
 $Comp
-L power:GND #PWR?
+L power:GND #PWR0128
 U 1 1 5CFBC187
 P 1600 2400
-AR Path="/5D1735E0/5CFBC187" Ref="#PWR?"  Part="1"
+AR Path="/5D1735E0/5CFBC187" Ref="#PWR0128"  Part="1"
 AR Path="/5D190D23/5CFBC187" Ref="#PWR?"  Part="1"
-F 0 "#PWR?" H 1600 2150 50  0001 C CNN
+F 0 "#PWR0128" H 1600 2150 50  0001 C CNN
 F 1 "GND" H 1605 2227 50  0000 C CNN
 F 2 "" H 1600 2400 50  0001 C CNN
@@
 	1600 2550 1450 2550
 $Comp
-L power:+3V3 #PWR?
+L power:+3V3 #PWR0129
 U 1 1 5CFBE976
 P 1800 2350
-AR Path="/5D1735E0/5CFBE976" Ref="#PWR?"  Part="1"
+AR Path="/5D1735E0/5CFBE976" Ref="#PWR0129"  Part="1"
 AR Path="/5D190D23/5CFBE976" Ref="#PWR?"  Part="1"
-F 0 "#PWR?" H 1800 2200 50  0001 C CNN
+F 0 "#PWR0129" H 1800 2200 50  0001 C CNN
 F 1 "+3V3" H 1815 2523 50  0000 C CNN
 F 2 "" H 1800 2350 50  0001 C CNN

Commit message: update,
Connections:
- net SCL: now also RN2.2 (R2.1); no longer RN2.1 (R1.1)
- net SDA: now also RN2.1 (R1.1); no longer RN2.2 (R2.1)
Changed lines of the file:
@@
 Text Label 4750 2250 2    50   ~ 0
 SDA
+Text Label 1950 2050 1    50   ~ 0
+SCL
 Text Label 1850 2050 1    50   ~ 0
-SCL
-Text Label 1950 2050 1    50   ~ 0
 SDA
 Wire Wire Line
+	1950 1700 1950 2050
+Wire Wire Line
 	1850 1700 1850 2050
-Wire Wire Line
-	1950 1700 1950 2050
 $Comp
 L Connector:Conn_01x06_Female J3
