File: hardware/power.sch (KiCad schematic (older format))
At the start: 8 parts, among them U11 AMS1117-3.3

Commit message: update,
Parts:
- D8: footprint LED_SMD:LED_0603_1608Metric_Pad1.05x0.95mm_HandSolder -> LED_SMD:LED_0805_2012Metric_Pad1.15x1.40mm_HandSolder
Other:
- moved on the sheet: D8, R19
Changed lines of the file:
@@
 L taobao-r:R102,0603 R?
 U 1 1 5C0C1058
-P 5100 1700
+P 5100 1350
 AR Path="/5C0BBB2B/5C0C1058" Ref="R?"  Part="1"
 AR Path="/5C0BFA48/5C0C1058" Ref="R?"  Part="1"
 AR Path="/5D194EE8/5C0C1058" Ref="R19"  Part="1"
-F 0 "R19" H 5200 1750 50  0000 L CNN
-F 1 "R102,0603" H 5200 1700 50  0000 L CNN
-F 2 "Resistor_SMD:R_0603_1608Metric_Pad1.05x0.95mm_HandSolder" H 5100 1700 50  0001 C CNN
-F 3 "~" H 5100 1700 50  0001 C CNN
-	1    5100 1700
+F 0 "R19" H 5200 1400 50  0000 L CNN
+F 1 "R102,0603" H 5200 1350 50  0000 L CNN
+F 2 "Resistor_SMD:R_0603_1608Metric_Pad1.05x0.95mm_HandSolder" H 5100 1350 50  0001 C CNN
+F 3 "~" H 5100 1350 50  0001 C CNN
+	1    5100 1350
 	1    0    0    -1
 $EndComp
@@
 L taobao-led:LED_GREEN,0603 D8
 U 1 1 5C0D46AA
-P 5100 1350
-F 0 "D8" V 5150 1250 50  0000 R CNN
-F 1 "3V3_HEALTHY" V 5100 1250 50  0000 R CNN
-F 2 "LED_SMD:LED_0603_1608Metric_Pad1.05x0.95mm_HandSolder" V 5100 1350 50  0001 C CNN
-F 3 "" V 5100 1350 50  0001 C CNN
-	1    5100 1350
+P 5100 1700
+F 0 "D8" V 5150 1600 50  0000 R CNN
+F 1 "3V3_HEALTHY" V 5100 1600 50  0000 R CNN
+F 2 "LED_SMD:LED_0805_2012Metric_Pad1.15x1.40mm_HandSolder" V 5100 1700 50  0001 C CNN
+F 3 "" V 5100 1700 50  0001 C CNN
+	1    5100 1700
 	0    -1   -1   0
 $EndComp
