File: hardware/ssd1306.sch (KiCad schematic (older format))
At the start: 2 parts, among them U10 SSD1306-OLED-I2C

Commit message: update,
Connections:
- net SCL: now also RN4.2 (R2.1); no longer RN4.1 (R1.1)
- net SDA: now also RN4.1 (R1.1); no longer RN4.2 (R2.1)
Changed lines of the file:
@@
 SDA
 Wire Wire Line
-	2200 2050 3050 2050
-Wire Wire Line
-	2200 2150 3150 2150
+	2200 2150 3050 2150
 $Comp
 L taobao-board:SSD1306-OLED-I2C U10
@@
 Connection ~ 3250 1200
 Wire Wire Line
-	3050 1850 3050 2050
-Connection ~ 3050 2050
+	3150 1850 3150 2050
 Wire Wire Line
-	3050 2050 3450 2050
-Wire Wire Line
-	3150 1850 3150 2150
-Connection ~ 3150 2150
-Wire Wire Line
-	3150 2150 3450 2150
+	3050 1850 3050 2150
 NoConn ~ 3250 1850
 NoConn ~ 3350 1850
+Wire Wire Line
+	2200 2050 3150 2050
+Connection ~ 3050 2150
+Wire Wire Line
+	3050 2150 3450 2150
+Connection ~ 3150 2050
+Wire Wire Line
+	3150 2050 3450 2050
 $EndSCHEMATC
