File: hardware/terminal.sch (KiCad schematic (older format))
At the start: 1 part

Commit message: update,
Parts:
- removed J?: I2C_HEADER, footprint-lib:CONN_I2C_SSD1306, symbol Connector:Conn_01x04_Female
- added RN5: RN_472,0603, Resistor_SMD:R_Array_Concave_4x0603, symbol taobao-rpack:RN_472,0603
- added U9: SSD1306-OLED-I2C, footprint-lib:CONN_I2C_SSD1306, symbol taobao-board:SSD1306-OLED-I2C
Connections:
- net +3V3: now also RN5.5 (R4.2), RN5.6 (R3.2), RN5.7 (R2.2), RN5.8 (R1.2), U9.VCC
- net GND: now also U9.GND
- net SCL: now also RN5.1 (R1.1), U9.SCL
- net SDA: now also RN5.2 (R2.1), U9.SDA
- no-connect marks 0 -> 2
Changed lines of the file:
@@
 EESchema Schematic File Version 4
-LIBS:PMS5003S_MOUNT-cache
-LIBS:bmp180_tryout-cache
+LIBS:cowin-tryout-cache
+LIBS:CH340T-tryout-cache
 EELAYER 29 0
 EELAYER END
 $Descr User 8500 5500
 encoding utf-8
-Sheet 6 8
+Sheet 6 12
 Title ""
 Date ""
@@
 $EndDescr
 $Comp
-L Connector:Conn_01x04_Female J?
-U 1 1 5D18F859
-P 1550 1250
-F 0 "J?" H 1442 1535 50  0000 C CNN
-F 1 "I2C_HEADER" H 1442 1444 50  0000 C CNN
-F 2 "footprint-lib:CONN_I2C_SSD1306" H 1550 1250 50  0001 C CNN
-F 3 "~" H 1550 1250 50  0001 C CNN
-	1    1550 1250
-	-1   0    0    -1
-$EndComp
-$Comp
-L power:+3V3 #PWR?
+L power:+3V3 #PWR0130
 U 1 1 5D18FCC7
-P 2050 950
-F 0 "#PWR?" H 2050 800 50  0001 C CNN
-F 1 "+3V3" H 2065 1123 50  0000 C CNN
-F 2 "" H 2050 950 50  0001 C CNN
-F 3 "" H 2050 950 50  0001 C CNN
-	1    2050 950
+P 2850 1900
+F 0 "#PWR0130" H 2850 1750 50  0001 C CNN
+F 1 "+3V3" H 2865 2073 50  0000 C CNN
+F 2 "" H 2850 1900 50  0001 C CNN
+F 3 "" H 2850 1900 50  0001 C CNN
+	1    2850 1900
 	1    0    0    -1
 $EndComp
 Wire Wire Line
-	1750 1150 2050 1150
+	2550 2100 2850 2100
 Wire Wire Line
-	2050 1150 2050 950
+	2850 2100 2850 1900
 $Comp
-L power:GND #PWR?
+L power:GND #PWR0131
 U 1 1 5D19015E
-P 2250 950
-F 0 "#PWR?" H 2250 700 50  0001 C CNN
-F 1 "GND" H 2255 777 50  0000 C CNN
-F 2 "" H 2250 950 50  0001 C CNN
-F 3 "" H 2250 950 50  0001 C CNN
-	1    2250 950
+P 3050 1900
+F 0 "#PWR0131" H 3050 1650 50  0001 C CNN
+F 1 "GND" H 3055 1727 50  0000 C CNN
+F 2 "" H 3050 1900 50  0001 C CNN
+F 3 "" H 3050 1900 50  0001 C CNN
+	1    3050 1900
 	-1   0    0    1
 $EndComp
 Wire Wire Line
-	1750 1250 2250 1250
+	2550 2200 3050 2200
 Wire Wire Line
-	2250 1250 2250 950
-Text HLabel 2450 1350 2    50   Input ~ 0
+	3050 2200 3050 1900
+Text HLabel 4400 2300 2    50   Input ~ 0
 SCL
-Text HLabel 2450 1450 2    50   Input ~ 0
+Text HLabel 4400 2400 2    50   Input ~ 0
 SDA
 Wire Wire Line
-	1750 1350 2450 1350
+	2550 2300 3450 2300
 Wire Wire Line
-	1750 1450 2450 1450
+	2550 2400 3550 2400
+$Comp
+L taobao-board:SSD1306-OLED-I2C U9
+U 1 1 5D18E076
+P 2350 2250
+F 0 "U9" H 2467 2765 50  0000 C CNN
+F 1 "SSD1306-OLED-I2C" H 2467 2674 50  0000 C CNN
+F 2 "footprint-lib:CONN_I2C_SSD1306" H 2350 2100 50  0001 C CNN
+F 3 "" H 2350 2100 50  0001 C CNN
+	1    2350 2250
+	-1   0    0    -1
+$EndComp
+Wire Wire Line
+	3550 1700 3550 1450
+Wire Wire Line
+	3450 1700 3450 1450
+Wire Wire Line
+	3450 1450 3550 1450
+$Comp
+L customized_power:+3V3 #PWR?
+U 1 1 5D1D9E25
+P 3450 1300
+AR Path="/5CF23B4E/5D1D9E25" Ref="#PWR?"  Part="1"
+AR Path="/5CF23C1A/5D1D9E25" Ref="#PWR?"  Part="1"
+AR Path="/5D19ABF9/5D1D9E25" Ref="#PWR?"  Part="1"
+AR Path="/5D192838/5D1D9E25" Ref="#PWR?"  Part="1"
+AR Path="/5D17F36B/5D1D9E25" Ref="#PWR0166"  Part="1"
+F 0 "#PWR0166" H 3450 1150 50  0001 C CNN
+F 1 "+3V3" H 3450 1500 50  0000 C CNN
+F 2 "" H 3450 1300 50  0001 C CNN
+F 3 "" H 3450 1300 50  0001 C CNN
+	1    3450 1300
+	-1   0    0    -1
+$EndComp
+Wire Wire Line
+	3450 1450 3450 1300
+Connection ~ 3450 1450
+$Comp
+L taobao-rpack:RN_472,0603 RN?
+U 1 1 5D1D9E2D
+P 3650 1900
+AR Path="/5CF23B4E/5D1D9E2D" Ref="RN?"  Part="1"
+AR Path="/5CF23C1A/5D1D9E2D" Ref="RN?"  Part="1"
+AR Path="/5D19ABF9/5D1D9E2D" Ref="RN?"  Part="1"
+AR Path="/5D192838/5D1D9E2D" Ref="RN?"  Part="1"
+AR Path="/5D17F36B/5D1D9E2D" Ref="RN5"  Part="1"
+F 0 "RN5" V 3233 1900 50  0000 C CNN
+F 1 "RN_472,0603" V 3324 1900 50  0000 C CNN
+F 2 "Resistor_SMD:R_Array_Concave_4x0603" V 3925 1900 50  0001 C CNN
+F 3 "~" H 3650 1900 50  0001 C CNN
+	1    3650 1900
+	1    0    0    -1
+$EndComp
+Wire Wire Line
+	3650 1700 3650 1450
+Wire Wire Line
+	3650 1450 3550 1450
+Connection ~ 3550 1450
+Wire Wire Line
+	3750 1700 3750 1450
+Wire Wire Line
+	3750 1450 3650 1450
+Connection ~ 3650 1450
+Wire Wire Line
+	3450 2100 3450 2300
+Wire Wire Line
+	3550 2100 3550 2400
+NoConn ~ 3650 2100
+NoConn ~ 3750 2100
+Connection ~ 3450 2300
+Wire Wire Line
+	3450 2300 4400 2300
+Connection ~ 3550 2400
+Wire Wire Line
+	3550 2400 4400 2400
 $EndSCHEMATC

Commit message: update,
Parts:
- added U?: TTL_TERMINAL, symbol taobao-board:TTL_TERMINAL
Connections:
- net GND: now also U?.1 (GND)
- new net RXD: U?.3 (RXD)
- new net TXD: U?.2 (TXD)
Changed lines of the file:
@@
 EESchema Schematic File Version 4
 LIBS:cowin-tryout-cache
-LIBS:CH340T-tryout-cache
 EELAYER 29 0
 EELAYER END
@@
 Wire Wire Line
 	3550 2400 4400 2400
+$Comp
+L taobao-board:TTL_TERMINAL U?
+U 1 1 5D14C894
+P 2350 3200
+F 0 "U?" H 2400 3600 50  0000 C CNN
+F 1 "TTL_TERMINAL" H 2400 3500 50  0000 C CNN
+F 2 "" H 2350 3150 50  0001 C CNN
+F 3 "" H 2350 3150 50  0001 C CNN
+	1    2350 3200
+	-1   0    0    -1
+$EndComp
+$Comp
+L power:GND #PWR?
+U 1 1 5D14D13E
+P 2850 2950
+F 0 "#PWR?" H 2850 2700 50  0001 C CNN
+F 1 "GND" H 2850 2750 50  0000 C CNN
+F 2 "" H 2850 2950 50  0001 C CNN
+F 3 "" H 2850 2950 50  0001 C CNN
+	1    2850 2950
+	-1   0    0    1
+$EndComp
+Wire Wire Line
+	2850 2950 2850 3100
+Wire Wire Line
+	2850 3100 2550 3100
+Wire Wire Line
+	2550 3200 3050 3200
+Wire Wire Line
+	2550 3300 3050 3300
+Text HLabel 3050 3200 2    50   Input ~ 0
+TXD
+Text HLabel 3050 3300 2    50   Input ~ 0
+RXD
 $EndSCHEMATC

Commit message: update,
Parts:
- gave numbers to parts that had none: 1
Changed lines of the file:
@@
 	3550 2400 4400 2400
 $Comp
-L taobao-board:TTL_TERMINAL U?
+L taobao-board:TTL_TERMINAL U14
 U 1 1 5D14C894
 P 2350 3200
-F 0 "U?" H 2400 3600 50  0000 C CNN
+F 0 "U14" H 2400 3600 50  0000 C CNN
 F 1 "TTL_TERMINAL" H 2400 3500 50  0000 C CNN
 F 2 "" H 2350 3150 50  0001 C CNN
@@
 $EndComp
 $Comp
-L power:GND #PWR?
+L power:GND #PWR0152
 U 1 1 5D14D13E
 P 2850 2950
-F 0 "#PWR?" H 2850 2700 50  0001 C CNN
+F 0 "#PWR0152" H 2850 2700 50  0001 C CNN
 F 1 "GND" H 2850 2750 50  0000 C CNN
 F 2 "" H 2850 2950 50  0001 C CNN

Commit message: update,
Parts:
- U14: footprint (none) -> Connector_PinHeader_1.27mm:PinHeader_1x03_P1.27mm_Vertical
Changed lines of the file:
@@
 EESchema Schematic File Version 4
 LIBS:cowin-tryout-cache
+LIBS:CH340T-tryout-cache
+LIBS:MCP73831-cache
 EELAYER 29 0
 EELAYER END
 $Descr User 8500 5500
 encoding utf-8
-Sheet 6 12
+Sheet 6 13
 Title ""
 Date ""
@@
 F 0 "U14" H 2400 3600 50  0000 C CNN
 F 1 "TTL_TERMINAL" H 2400 3500 50  0000 C CNN
-F 2 "" H 2350 3150 50  0001 C CNN
+F 2 "Connector_PinHeader_1.27mm:PinHeader_1x03_P1.27mm_Vertical" H 2350 3150 50  0001 C CNN
 F 3 "" H 2350 3150 50  0001 C CNN
 	1    2350 3200

Commit message: update,
Connections:
- net SCL: now also RN5.2 (R2.1); no longer RN5.1 (R1.1)
- net SDA: now also RN5.1 (R1.1); no longer RN5.2 (R2.1)
Changed lines of the file:
@@
 SDA
 Wire Wire Line
-	2550 2300 3450 2300
-Wire Wire Line
-	2550 2400 3550 2400
+	2550 2400 3450 2400
 $Comp
 L taobao-board:SSD1306-OLED-I2C U9
@@
 Connection ~ 3650 1450
 Wire Wire Line
-	3450 2100 3450 2300
+	3550 2100 3550 2300
 Wire Wire Line
-	3550 2100 3550 2400
+	3450 2100 3450 2400
 NoConn ~ 3650 2100
 NoConn ~ 3750 2100
-Connection ~ 3450 2300
-Wire Wire Line
-	3450 2300 4400 2300
-Connection ~ 3550 2400
-Wire Wire Line
-	3550 2400 4400 2400
 $Comp
 L taobao-board:TTL_TERMINAL U14
@@
 Text HLabel 3050 3300 2    50   Input ~ 0
 RXD
+Wire Wire Line
+	2550 2300 3550 2300
+Connection ~ 3450 2400
+Wire Wire Line
+	3450 2400 4400 2400
+Connection ~ 3550 2300
+Wire Wire Line
+	3550 2300 4400 2300
 $EndSCHEMATC
