File: hardware/MCP73831.sch (KiCad schematic (older format))
At the start: 12 parts, among them J4 PWR_SRC, J5 5V_OUT, J8 BAT, U16 MCP73831

Commit message: update,
Parts:
- D9: footprint footprint-lib:LED_0603_1608Metric -> LED_SMD:LED_0805_2012Metric_Pad1.15x1.40mm_HandSolder
Changed lines of the file:
@@
 F 0 "D9" H 1350 2400 50  0000 C CNN
 F 1 "CHARGING" H 1350 2500 50  0000 C CNN
-F 2 "footprint-lib:LED_0603_1608Metric" V 1350 2250 50  0001 C CNN
+F 2 "LED_SMD:LED_0805_2012Metric_Pad1.15x1.40mm_HandSolder" V 1350 2250 50  0001 C CNN
 F 3 "" V 1350 2250 50  0001 C CNN
 	1    1350 2250
