File: hardware/cowin-tryout.kicad_pcb (KiCad board)
At the start: 2 copper layers, 63 x 52 mm, 78 parts, among them J1 BMP180_HEADER, J2 CONN_PMS, J3 SHT3x_HEADER, J7 DEBUG_HEADER, Q1 SS9013_J3, Q2 SS9013_J3, SW1 FLASH_BUTTON, SW2 SW_RESET,2_leg,SMD, U1 BMP180, U10 SSD1306-OLED-I2C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

Commit message: update,
Parts:
- D8: footprint LED_SMD:LED_0603_1608Metric_Pad1.05x0.95mm_HandSolder -> LED_SMD:LED_0805_2012Metric_Pad1.15x1.40mm_HandSolder
- J2, R19: moved to B.Cu
- moved C19 25.0 mm to (56.8, 67.0), turned to 270 degrees
- moved J7 23.9 mm to (113.3, 61.2)
- moved RN1 19.4 mm to (61.5, 67.2), turned to 270 degrees
- moved C1 18.5 mm to (56.8, 72.0), turned to 270 degrees
- moved J2 18.0 mm to (81.0, 55.5)
- moved C5 16.9 mm to (57.5, 82.0), turned to 0 degrees
- moved U1 15.0 mm to (60.8, 71.5), turned to 180 degrees
- moved JP2 13.8 mm to (67.0, 80.0), turned to 0 degrees
- moved U4 12.0 mm to (57.8, 78.8), turned to 90 degrees
- moved JP1 11.6 mm to (67.0, 77.0), turned to 0 degrees
- moved U11 11.5 mm to (81.0, 70.8), turned to 180 degrees
- moved J3 11.0 mm to (71.0, 81.0), turned to 180 degrees
- moved RN5 10.9 mm to (108.0, 55.2)
- moved R19 10.9 mm to (89.4, 55.5), turned to 270 degrees
- moved D8 8.83 mm to (89.4, 55.6), turned to 270 degrees
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Connections:
- D5 pad 2: Net-(D5-Pad2) -> (no net)
- D8 pad 1: Net-(D8-Pad1) -> GND
- D8 pad 2: +3V3 -> Net-(D8-Pad2)
- J2 pad 7: Net-(J2-Pad7) -> (no net)
- J2 pad 8: Net-(J2-Pad8) -> (no net)
- R19 pad 1: Net-(D8-Pad1) -> +3V3
- R19 pad 2: GND -> Net-(D8-Pad2)
- RN1 pad 3: Net-(RN1-Pad3) -> (no net)
- RN1 pad 4: Net-(RN1-Pad4) -> (no net)
- RN1 pad 5: Net-(RN1-Pad5) -> (no net)
- RN1 pad 6: Net-(RN1-Pad6) -> (no net)
- RN4 pad 3: Net-(RN4-Pad3) -> (no net)
- RN4 pad 4: Net-(RN4-Pad4) -> (no net)
- RN5 pad 3: Net-(RN5-Pad3) -> (no net)
- RN5 pad 4: Net-(RN5-Pad4) -> (no net)
- U1 pad 1: Net-(U1-Pad1) -> (no net)
- U1 pad 4: Net-(U1-Pad4) -> (no net)
- U2 pad 1: Net-(U2-Pad1) -> (no net)
- U2 pad 11: Net-(U2-Pad11) -> (no net)
- U2 pad 12: Net-(U2-Pad12) -> (no net)
- U2 pad 2: Net-(U2-Pad2) -> (no net)
- U2 pad 3: Net-(U2-Pad3) -> (no net)
- U2 pad 6: Net-(U2-Pad6) -> (no net)
- U2 pad 9: Net-(U2-Pad9) -> (no net)
- U6 pad 10: /esp-12e/SPI_MISO -> (no net)
- U6 pad 11: /esp-12e/GPIO9 -> (no net)
- U6 pad 12: /esp-12e/GPIO10 -> (no net)
- U6 pad 13: /esp-12e/SPI_INT -> (no net)
- U6 pad 14: /esp-12e/SPI_CLK -> (no net)
- U6 pad 7: /esp-12e/GPIO13 -> (no net)
- U6 pad 9: /esp-12e/SPI_MOSI -> (no net)
- U7 pad 11: /esp-12e/usb_to_uart/CTS -> (no net)
- U7 pad 12: /esp-12e/usb_to_uart/DSR -> (no net)
- U7 pad 13: /esp-12e/usb_to_uart/RI -> (no net)
- U7 pad 14: /esp-12e/usb_to_uart/DCD -> (no net)
- U7 pad 17: Net-(U7-Pad17) -> (no net)
- U7 pad 20: Net-(U7-Pad20) -> (no net)
- U8 pad 4: Net-(U8-Pad4) -> (no net)

Commit message: update,
Parts:
- added C20: C106,0603, Capacitor_SMD:C_0603_1608Metric_Pad1.05x0.95mm_HandSolder, F.Cu at (80.5, 64.5)
- added C21: C106,0603, Capacitor_SMD:C_0603_1608Metric_Pad1.05x0.95mm_HandSolder, F.Cu at (92.0, 68.0)
- added D6: D_1N4148_T4, Diode_SMD:D_SOD-123, F.Cu at (87.0, 60.5)
- added D9: CHARGING, footprint-lib:LED_0805_2012Metric, F.Cu at (92.0, 55.5)
- added J8: BAT, Connector_PinHeader_2.54mm:PinHeader_1x02_P2.54mm_Vertical, F.Cu at (114.5, 74.5)
- added JP4: 5V_EN, Jumper:SolderJumper-2_P1.3mm_Open_RoundedPad1.0x1.5mm, F.Cu at (91.5, 60.5)
- added JP6: OUT_EN, Jumper:SolderJumper-2_P1.3mm_Open_RoundedPad1.0x1.5mm, F.Cu at (91.5, 64.5)
- added R11: R102,0603, Resistor_SMD:R_0603_1608Metric_Pad1.05x0.95mm_HandSolder, B.Cu at (92.0, 55.5)
- added R20: R103,0603, Resistor_SMD:R_0603_1608Metric_Pad1.05x0.95mm_HandSolder, F.Cu at (83.0, 64.5)
- added U12: DESIGNED_IN_HONG_KONG, footprint-lib:DESIGNED_IN_HONG_KONG, F.Cu at (170.3, 74.2)
- added U13: GITHUB_ADDRESS, footprint-lib:GITHUB_ADDRESS, F.Cu at (171.8, 74.2)
- added U14: TTL_TERMINAL, Connector_PinHeader_1.27mm:PinHeader_1x03_P1.27mm_Vertical, F.Cu at (88.0, 100.0)
- added U15: BOARD_REVISION, footprint-lib:BOARD_REVISION, F.Cu at (173.3, 74.2)
- added U16: MCP73831, footprint-lib:MCP73831_SOT23_5, F.Cu at (86.5, 64.5)
- D1, D2, D8: footprint LED_SMD:LED_0805_2012Metric_Pad1.15x1.40mm_HandSolder -> footprint-lib:LED_0805_2012Metric
- moved U5 9.93 mm to (81.5, 93.5), turned to 0 degrees
- moved U11 2.68 mm to (79.5, 73.0)
- moved C18 2.01 mm to (90.5, 75.5)
- moved C17 2.00 mm to (87.5, 75.5)
- moved JP5 1.83 mm to (87.0, 71.0)
- moved C2 1.50 mm to (58.8, 87.7)
- moved C3 1.50 mm to (58.8, 85.9)
- moved JP3 1.50 mm to (91.0, 71.0)
- moved R1 1.50 mm to (62.6, 87.7)
- moved U2 1.50 mm to (59.3, 91.0)
Connections:
- U8 pad 1: +5V -> VBUS
Routing:
- net +3V3: track 0.00 -> 257.4 mm, vias 0 -> 4
- net +5V: track 0.00 -> 163.1 mm, vias 0 -> 1
- net /SDA: track 0.00 -> 143.2 mm, vias 0 -> 1
- net /SCL: track 0.00 -> 121.3 mm, vias 0 -> 4
- net /TXD: track 0.00 -> 111.8 mm
- net /RXD: track 0.00 -> 86.5 mm
- net /GPIO12: track 0.00 -> 67.3 mm, vias 0 -> 1
- net /esp-12e/nRST: track 0.00 -> 59.6 mm, vias 0 -> 2
- net /esp-12e/ADC: track 0.00 -> 52.4 mm, vias 0 -> 2
- net /sunlight_uv/EN: track 0.00 -> 52.0 mm
- net Net-(R15-Pad2): track 0.00 -> 50.4 mm
- net /esp-12e/GPIO0: track 0.00 -> 49.9 mm, vias 0 -> 1
- net Net-(C18-Pad1): track 0.00 -> 48.9 mm
- net /esp-12e/GPIO2: track 0.00 -> 48.6 mm, vias 0 -> 1
- net /esp-12e/usb_to_uart/RXD0: track 0.00 -> 43.9 mm, vias 0 -> 2
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
Commit message: update,
Parts:
- removed TP1: TP_RXD, TestPoint:TestPoint_Pad_1.0x1.0mm
- removed TP2: TP_TXD, TestPoint:TestPoint_Pad_1.0x1.0mm
- added C22: C106,0805, Capacitor_SMD:C_0805_2012Metric_Pad1.15x1.40mm_HandSolder, F.Cu at (73.1, 63.6)
- added RN3: RN_472,0603, Resistor_SMD:R_Array_Concave_4x0603, F.Cu at (79.1, 69.0)
- added U17: 24C02_SOIC8, footprint-lib:24Cxx_SOIC8, F.Cu at (73.1, 68.0)
- D1, D2, D8: footprint footprint-lib:LED_0805_2012Metric -> LED_SMD:LED_0805_2012Metric_Pad1.15x1.40mm_HandSolder
- D9: footprint footprint-lib:LED_0805_2012Metric -> footprint-lib:LED_0603_1608Metric
- moved U15 12.4 mm to (161.0, 73.0)
- moved U12 11.8 mm to (163.9, 84.0)
- moved U13 8.75 mm to (164.2, 78.5)
- moved R12 5.51 mm to (86.0, 94.4), turned to 270 degrees
- moved U11 3.03 mm to (79.9, 76.0)
Routing:
- net /SCL: track 121.3 -> 167.3 mm, vias 4 -> 6
- net GND: track 9.36 -> 30.8 mm, vias 4 -> 9
- net +3V3: track 257.4 -> 276.1 mm, vias 4 -> 6
- net /SDA: track 143.2 -> 153.2 mm, vias 1 -> 2
- net /RXD: track 86.5 -> 76.9 mm, vias 0 -> 1
- net /TXD: track 111.8 -> 103.4 mm, vias 0 -> 3
- net Net-(C18-Pad1): track 48.9 -> 55.1 mm
- net /esp-12e/usb_to_uart/RXD0: track 43.9 -> 38.0 mm
- net +5V: track 163.1 -> 168.6 mm
- net Net-(C17-Pad1): track 12.6 -> 10.6 mm
- net /sunlight_uv/EN: track 52.0 -> 54.0 mm
- net /esp-12e/nRST: track 59.6 -> 61.5 mm
- net Vbat: track 39.0 -> 40.7 mm
- net /esp-12e/GPIO0: track 49.9 -> 51.4 mm
- net Net-(D3-Pad4): track 7.52 -> 6.21 mm
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
Commit message: update,
Parts:
- moved JP1 10.3 mm to (58.5, 82.9)
- moved C5 6.24 mm to (62.8, 85.3), turned to 180 degrees
- moved JP2 5.10 mm to (62.8, 82.9)
- moved J1 4.64 mm to (66.6, 68.7), turned to 0 degrees
- moved D7 4.39 mm to (113.5, 91.2)
- moved R13 4.27 mm to (115.2, 91.2), turned to 90 degrees
- moved R8 4.26 mm to (111.5, 94.9)
- moved RN2 3.91 mm to (66.2, 77.5), turned to 180 degrees
- moved R12 3.02 mm to (88.5, 92.7), turned to 180 degrees
- moved U4 2.84 mm to (60.3, 77.5)
- moved U14 2.67 mm to (88.6, 97.4), turned to 180 degrees
- moved R6 2.10 mm to (86.8, 87.2)
- moved RN3 1.63 mm to (80.2, 70.2)
- moved R7 1.50 mm to (86.8, 85.0)
- moved U1 0.75 mm to (61.2, 72.1), turned to 90 degrees
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Connections:
- RN1 pad 1: /SCL -> /SDA
- RN1 pad 2: /SDA -> /SCL
- RN2 pad 1: /SCL -> /SDA
- RN2 pad 2: /SDA -> /SCL
- RN4 pad 1: /SCL -> /SDA
- RN4 pad 2: /SDA -> /SCL
- RN5 pad 1: /SCL -> /SDA
- RN5 pad 2: /SDA -> /SCL
Routing:
- net +3V3: track 276.1 -> 22.9 mm, vias 6 -> 2
- net +5V: track 168.6 -> 0.00 mm, vias 1 -> 0
- net /TXD: track 103.4 -> 4.85 mm, vias 3 -> 0
- net /GPIO12: track 67.3 -> 0.00 mm, vias 1 -> 0
- net /esp-12e/nRST: track 61.5 -> 0.00 mm, vias 2 -> 0
- net Net-(C18-Pad1): track 55.1 -> 0.00 mm
- net /RXD: track 76.9 -> 22.7 mm, vias 1 -> 0
- net /sunlight_uv/EN: track 54.0 -> 0.00 mm
- net /esp-12e/ADC: track 52.5 -> 0.00 mm, vias 4 -> 0
- net /esp-12e/GPIO0: track 51.4 -> 0.00 mm, vias 1 -> 0
- net Net-(R15-Pad2): track 50.4 -> 0.00 mm
- net /esp-12e/GPIO2: track 48.6 -> 0.00 mm, vias 1 -> 0
- net Vbat: track 40.7 -> 0.00 mm
- net /esp-12e/usb_to_uart/RXD0: track 38.0 -> 0.00 mm, vias 2 -> 0
- net /SCL: track 167.3 -> 133.8 mm, vias 6 -> 5
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Other:
- net class 300mA added: clearance 0.2, trace_width 0.3, via_dia 0.8, via_drill 0.4
- net class GND added: clearance 0.2, trace_width 0.5, via_dia 0.8, via_drill 0.4

Commit message: update,
Parts:
- moved J7 11.2 mm to (113.6, 72.4)
- moved C11 2.86 mm to (114.9, 64.9)
- moved U8 2.80 mm to (115.3, 64.9)
- moved J8 1.92 mm to (113.6, 76.2), turned to 90 degrees
- moved C14 1.50 mm to (109.4, 67.6)
- moved U2 1.01 mm to (59.3, 92.0)
- moved RN4 0.55 mm to (108.0, 59.2)
Connections:
- U7 pad 10: Net-(C16-Pad1) -> Net-(C15-Pad1)
- U7 pad 9: Net-(C15-Pad1) -> Net-(C16-Pad1)
Routing:
- net +3V3: track 22.9 -> 297.7 mm, vias 2 -> 9
- net +5V: track 0.00 -> 174.4 mm, vias 0 -> 7
- net /esp-12e/nRST: track 0.00 -> 139.3 mm, vias 0 -> 9
- net Net-(C18-Pad1): track 0.00 -> 99.1 mm, vias 0 -> 6
- net GND: track 0.00 -> 97.3 mm, vias 0 -> 37
- net /TXD: track 4.85 -> 99.9 mm, vias 0 -> 2
- net /GPIO12: track 0.00 -> 80.9 mm, vias 0 -> 4
- net Net-(R15-Pad2): track 0.00 -> 66.2 mm, vias 0 -> 3
- net /RXD: track 22.7 -> 87.2 mm
- net /esp-12e/ADC: track 0.00 -> 62.4 mm, vias 0 -> 2
- net /esp-12e/GPIO0: track 0.00 -> 60.7 mm, vias 0 -> 3
- net /sunlight_uv/EN: track 0.00 -> 55.2 mm, vias 0 -> 2
- net /esp-12e/usb_to_uart/RXD0: track 0.00 -> 53.1 mm, vias 0 -> 2
- net Vbat: track 0.00 -> 42.5 mm, vias 0 -> 7
- net /esp-12e/GPIO2: track 0.00 -> 41.7 mm, vias 0 -> 3
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
Commit message: update,
Parts:
- added J9: DHT22_HEADER, Connector_PinHeader_2.54mm:PinHeader_1x03_P2.54mm_Vertical, F.Cu at (87.9, 98.0)
- added R21: R103,0603, Resistor_SMD:R_0603_1608Metric_Pad1.05x0.95mm_HandSolder, B.Cu at (81.9, 95.2)
- D9: footprint footprint-lib:LED_0603_1608Metric -> LED_SMD:LED_0805_2012Metric_Pad1.15x1.40mm_HandSolder
- J8, U5: moved to B.Cu
- Q1, R18: moved to F.Cu
- R4, R5: footprint Resistor_SMD:R_0805_2012Metric_Pad1.15x1.40mm_HandSolder -> Resistor_SMD:R_0603_1608Metric_Pad1.05x0.95mm_HandSolder
- moved U5 7.50 mm to (81.8, 101.0)
- moved R12 5.23 mm to (84.7, 96.3), turned to 270 degrees
- moved U14 4.37 mm to (87.1, 93.3), turned to 90 degrees
- moved R18 4.05 mm to (111.4, 85.0), turned to 90 degrees
- moved Q1 4.05 mm to (114.1, 85.0), turned to 270 degrees
- moved J8 2.40 mm to (113.6, 78.6), turned to 0 degrees
- moved C5 1.70 mm to (62.8, 87.0)
- moved R1 1.30 mm to (62.6, 89.0)
- moved JP2 0.62 mm to (63.0, 83.5)
- moved J7 0.60 mm to (113.6, 71.8)
- moved R5 0.15 mm to (84.2, 55.5)
- moved D9 0.08 mm to (92.0, 55.6)
- moved R4 0.08 mm to (86.9, 55.5)
- moved D2 0.07 mm to (84.2, 55.6)
Connections:
- U6 pad 7: (no net) -> /DHT_OUT
Routing:
- net /DHT_OUT: track 0.00 -> 47.3 mm, vias 0 -> 2
- net GND: track 97.3 -> 116.1 mm, vias 37 -> 46
- net Net-(D1-Pad2): track 16.1 -> 0.00 mm, vias 3 -> 1
- net /esp-12e/usb_to_uart/RTS: track 13.2 -> 29.1 mm, vias 1 -> 2
- net /RXD: track 87.2 -> 77.6 mm, vias 0 -> 1
- net Net-(D3-Pad4): track 7.52 -> 1.35 mm, vias 0 -> 1
- net /esp-12e/GPIO0: track 60.7 -> 66.7 mm
- net /esp-12e/nRST: track 139.3 -> 144.6 mm, vias 9 -> 11
- net +3V3: track 297.7 -> 302.8 mm, vias 9 -> 11
- net Vbat: track 42.5 -> 37.5 mm
- net /esp-12e/usb_to_uart/RXD0: track 53.1 -> 57.1 mm
- net +5V: track 174.4 -> 178.3 mm, vias 7 -> 9
- net /esp-12e/usb_to_uart/DTR: track 21.2 -> 17.5 mm
- net Net-(D2-Pad2): track 3.07 -> 0.00 mm
- net Net-(JP1-Pad2): track 17.8 -> 20.5 mm
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
Commit message: update,
Parts:
- R4, R5: footprint Resistor_SMD:R_0603_1608Metric_Pad1.05x0.95mm_HandSolder -> Resistor_SMD:R_0805_2012Metric_Pad1.15x1.40mm_HandSolder
- moved C4 17.3 mm to (79.8, 58.3), turned to 180 degrees
- turned R11 to 90 degrees
Connections:
- RN1 pad 5: (no net) -> +3V3
- RN1 pad 6: (no net) -> +3V3
Routing:
- net +3V3: track 302.8 -> 343.2 mm, vias 11 -> 13
- net Net-(D9-Pad1): track 25.7 -> 0.02 mm, vias 3 -> 1
- net +5V: track 178.3 -> 159.8 mm
- net /RXD: track 77.6 -> 91.1 mm
- net GND: track 116.1 -> 126.8 mm, vias 46 -> 51
- net Net-(R11-Pad1): track 17.7 -> 15.2 mm, vias 1 -> 3
- net Net-(D9-Pad2): track 13.5 -> 15.1 mm
- net /TXD: track 102.0 -> 103.6 mm
- net Vbat: track 37.5 -> 38.4 mm
- net /GPIO12: track 79.7 -> 80.5 mm
- net Net-(C18-Pad1): track 97.2 -> 96.6 mm
- net /pm2_5/SEN_RESET: track 12.4 -> 11.9 mm

Commit message: update,
Parts:
- R4, R5: footprint Resistor_SMD:R_0805_2012Metric_Pad1.15x1.40mm_HandSolder -> Resistor_SMD:R_0603_1608Metric_Pad1.05x0.95mm_HandSolder
- moved R21 30.5 mm to (112.0, 100.0), turned to 270 degrees
- moved J9 27.6 mm to (115.5, 96.5)
- moved U14 15.7 mm to (87.5, 109.0), turned to 180 degrees
- moved R12 6.75 mm to (85.5, 103.0), turned to 0 degrees
- moved U6 6.25 mm to (101.0, 99.0)
- moved C6 6.20 mm to (80.0, 103.0)
- moved D5 6.13 mm to (65.0, 107.2)
- moved D3 6.13 mm to (82.0, 107.2)
- moved U5 6.13 mm to (82.0, 107.1)
- moved D4 6.12 mm to (73.5, 107.2)
- moved C2 6.00 mm to (58.8, 93.7)
- moved C3 6.00 mm to (58.8, 91.9)
- moved C5 6.00 mm to (62.8, 93.0)
- moved C9 6.00 mm to (80.0, 93.8)
- moved H1 6.00 mm to (58.0, 108.0)
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Routing:
- net +3V3: track 343.2 -> 0.00 mm, vias 13 -> 0
- net +5V: track 159.8 -> 0.00 mm, vias 9 -> 0
- net /esp-12e/nRST: track 144.6 -> 0.00 mm, vias 11 -> 0
- net GND: track 126.8 -> 7.19 mm, vias 51 -> 1
- net Net-(C18-Pad1): track 96.6 -> 0.00 mm, vias 6 -> 0
- net /GPIO12: track 80.5 -> 0.00 mm, vias 4 -> 0
- net /RXD: track 91.1 -> 20.1 mm, vias 1 -> 0
- net Net-(R15-Pad2): track 68.2 -> 0.00 mm, vias 3 -> 0
- net /esp-12e/GPIO0: track 66.7 -> 0.00 mm, vias 3 -> 0
- net /esp-12e/ADC: track 62.8 -> 0.00 mm, vias 4 -> 0
- net /sunlight_uv/EN: track 54.8 -> 0.00 mm, vias 2 -> 0
- net /DHT_OUT: track 46.9 -> 0.00 mm, vias 2 -> 0
- net /esp-12e/GPIO2: track 42.1 -> 0.00 mm, vias 3 -> 0
- net Vbat: track 38.4 -> 0.00 mm, vias 7 -> 0
- net /TXD: track 103.6 -> 68.6 mm, vias 2 -> 3
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- removed copper zone on B.Cu, net GND
- removed copper zone on F.Cu, net GND
Other:
- board size 63 x 52 mm -> 63 x 58 mm
