File: hardware/cowin-tryout.kicad_pcb (KiCad board)
At the start: 2 copper layers, 63 x 58 mm, 95 parts, among them J1 BMP180_HEADER, J2 CONN_PMS, J3 SHT3x_HEADER, J7 DEBUG_HEADER, J8 BAT, J9 DHT22_HEADER, Q1 SS9013_J3, Q2 SS9013_J3, SW1 FLASH_BUTTON, SW2 SW_RESET,2_leg,SMD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

Commit message: update,
Parts:
- added J10: USB_DBG, Connector_PinHeader_2.54mm:PinHeader_1x05_P2.54mm_Vertical, F.Cu at (110.0, 68.3)
- moved U13 69.8 mm to (101.0, 107.9)
- moved U15 68.6 mm to (101.0, 106.3)
- moved U12 68.0 mm to (101.0, 109.6)
- moved R2 8.36 mm to (75.9, 59.4)
- moved R3 7.09 mm to (68.3, 59.4)
- moved C1 5.25 mm to (61.0, 72.1), turned to 180 degrees
- moved C4 1.78 mm to (78.5, 59.4), turned to 90 degrees
- moved RN4 1.65 mm to (106.3, 60.7)
- moved RN5 1.65 mm to (106.3, 56.0)
- moved U7 1.30 mm to (103.7, 72.0)
- moved C15 1.20 mm to (96.8, 67.9)
- moved C16 1.20 mm to (96.8, 75.1)
- moved Y1 1.20 mm to (96.8, 71.5)
- moved JP4 0.78 mm to (90.8, 60.1)
- moved D6 0.76 mm to (86.2, 60.4)
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Connections:
- net Net-(U7-Pad6) renamed /esp-12e/usb_to_uart/USB_P
- net Net-(U7-Pad7) renamed /esp-12e/usb_to_uart/USB_N
- D5 pad 2: (no net) -> Net-(D5-Pad2)
- J2 pad 7: (no net) -> Net-(J2-Pad7)
- J2 pad 8: (no net) -> Net-(J2-Pad8)
- RN1 pad 3: (no net) -> Net-(RN1-Pad3)
- RN1 pad 4: (no net) -> Net-(RN1-Pad4)
- RN3 pad 3: (no net) -> Net-(RN3-Pad3)
- RN3 pad 4: (no net) -> Net-(RN3-Pad4)
- RN3 pad 5: (no net) -> Net-(RN3-Pad5)
- RN3 pad 6: (no net) -> Net-(RN3-Pad6)
- RN4 pad 3: (no net) -> Net-(RN4-Pad3)
- RN4 pad 4: (no net) -> Net-(RN4-Pad4)
- RN5 pad 3: (no net) -> Net-(RN5-Pad3)
- RN5 pad 4: (no net) -> Net-(RN5-Pad4)
- U1 pad 1: (no net) -> Net-(U1-Pad1)
- U1 pad 4: (no net) -> Net-(U1-Pad4)
- U2 pad 1: (no net) -> Net-(U2-Pad1)
- U2 pad 11: (no net) -> Net-(U2-Pad11)
- U2 pad 12: (no net) -> Net-(U2-Pad12)
- U2 pad 2: (no net) -> Net-(U2-Pad2)
- U2 pad 3: (no net) -> Net-(U2-Pad3)
- U2 pad 6: (no net) -> Net-(U2-Pad6)
- U2 pad 9: (no net) -> Net-(U2-Pad9)
- U6 pad 10: (no net) -> /esp-12e/SPI_MISO
- U6 pad 11: (no net) -> /esp-12e/GPIO9
- U6 pad 12: (no net) -> /esp-12e/GPIO10
- U6 pad 13: (no net) -> /esp-12e/SPI_INT
- U6 pad 14: (no net) -> /esp-12e/SPI_CLK
- U6 pad 9: (no net) -> /esp-12e/SPI_MOSI
- U7 pad 11: (no net) -> /esp-12e/usb_to_uart/CTS
- U7 pad 12: (no net) -> /esp-12e/usb_to_uart/DSR
- U7 pad 13: (no net) -> /esp-12e/usb_to_uart/RI
- U7 pad 14: (no net) -> /esp-12e/usb_to_uart/DCD
- U7 pad 17: (no net) -> Net-(U7-Pad17)
- U7 pad 20: (no net) -> Net-(U7-Pad20)
- U8 pad 4: (no net) -> /esp-12e/usb_to_uart/ID
Routing:
- net GND: track 7.19 -> 399.9 mm, vias 1 -> 54
- net +3V3: track 0.00 -> 302.8 mm, vias 0 -> 15
- net +5V: track 0.00 -> 198.2 mm, vias 0 -> 10
- net Net-(C18-Pad1): track 0.00 -> 80.5 mm, vias 0 -> 4
- net /RXD: track 20.1 -> 99.5 mm
- net /esp-12e/nRST: track 0.00 -> 72.9 mm, vias 0 -> 5
- net /GPIO12: track 0.00 -> 69.3 mm, vias 0 -> 3
- net /esp-12e/GPIO0: track 0.00 -> 62.6 mm, vias 0 -> 3
- net /sunlight_uv/EN: track 0.00 -> 60.0 mm, vias 0 -> 4
- net /esp-12e/ADC: track 0.00 -> 53.7 mm, vias 0 -> 3
- net Net-(R15-Pad2): track 0.00 -> 52.5 mm, vias 0 -> 4
- net /esp-12e/GPIO2: track 0.00 -> 50.0 mm, vias 0 -> 2
- net VBUS: track 0.00 -> 41.2 mm, vias 0 -> 1
- net Vbat: track 0.00 -> 38.7 mm, vias 0 -> 4
- net /TXD: track 68.6 -> 98.6 mm, vias 3 -> 5
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- added copper zone on B.Cu, net GND
- added copper zone on F.Cu, net GND
Other:
- net class 300mA: trace_width 0.3 -> 0.4
- net class GND: trace_width 0.5 -> 0.6

Commit message: update,
Parts:
- removed D2: 3V3_HEALTHY, LED_SMD:LED_0805_2012Metric_Pad1.15x1.40mm_HandSolder
- removed R5: R102, Resistor_SMD:R_0603_1608Metric_Pad1.05x0.95mm_HandSolder
- moved D1 2.00 mm to (84.9, 55.6)
- moved R4 2.00 mm to (84.9, 55.5)
- moved D8 1.50 mm to (87.9, 55.6)
- moved R19 1.50 mm to (87.9, 55.5)
- moved D9 1.00 mm to (91.0, 55.6)
- moved R11 1.00 mm to (91.0, 55.5)
Connections:
- D5 pad 2: Net-(D5-Pad2) -> (no net)
- J2 pad 7: Net-(J2-Pad7) -> (no net)
- J2 pad 8: Net-(J2-Pad8) -> (no net)
- RN1 pad 3: Net-(RN1-Pad3) -> (no net)
- RN1 pad 4: Net-(RN1-Pad4) -> (no net)
- RN3 pad 3: Net-(RN3-Pad3) -> (no net)
- RN3 pad 4: Net-(RN3-Pad4) -> (no net)
- RN3 pad 5: Net-(RN3-Pad5) -> (no net)
- RN3 pad 6: Net-(RN3-Pad6) -> (no net)
- RN4 pad 3: Net-(RN4-Pad3) -> (no net)
- RN4 pad 4: Net-(RN4-Pad4) -> (no net)
- RN5 pad 3: Net-(RN5-Pad3) -> (no net)
- RN5 pad 4: Net-(RN5-Pad4) -> (no net)
- U1 pad 1: Net-(U1-Pad1) -> (no net)
- U1 pad 4: Net-(U1-Pad4) -> (no net)
- U2 pad 1: Net-(U2-Pad1) -> (no net)
- U2 pad 11: Net-(U2-Pad11) -> (no net)
- U2 pad 12: Net-(U2-Pad12) -> (no net)
- U2 pad 2: Net-(U2-Pad2) -> (no net)
- U2 pad 3: Net-(U2-Pad3) -> (no net)
- U2 pad 6: Net-(U2-Pad6) -> (no net)
- U2 pad 9: Net-(U2-Pad9) -> (no net)
- U6 pad 10: /esp-12e/SPI_MISO -> (no net)
- U6 pad 11: /esp-12e/GPIO9 -> (no net)
- U6 pad 12: /esp-12e/GPIO10 -> (no net)
- U6 pad 13: /esp-12e/SPI_INT -> (no net)
- U6 pad 14: /esp-12e/SPI_CLK -> (no net)
- U6 pad 9: /esp-12e/SPI_MOSI -> (no net)
- U7 pad 11: /esp-12e/usb_to_uart/CTS -> (no net)
- U7 pad 12: /esp-12e/usb_to_uart/DSR -> (no net)
- U7 pad 13: /esp-12e/usb_to_uart/RI -> (no net)
- U7 pad 14: /esp-12e/usb_to_uart/DCD -> (no net)
- U7 pad 17: Net-(U7-Pad17) -> (no net)
- U7 pad 20: Net-(U7-Pad20) -> (no net)
Routing:
- net GND: track 399.9 -> 405.3 mm
- net VBUS: track 41.2 -> 37.8 mm, vias 1 -> 4
- net Net-(D9-Pad1): track 3.02 -> 0.00 mm
- net Net-(D3-Pad4): track 5.82 -> 3.02 mm
- net Net-(D2-Pad2): track 2.64 -> 0.00 mm, vias 1 -> 0
- net Net-(D1-Pad2): track 2.62 -> 0.00 mm
- net Net-(D8-Pad2): track 2.58 -> 0.00 mm
- net Net-(D9-Pad2): track 9.92 -> 12.3 mm
- net /sunlight_uv/EN: track 60.0 -> 62.0 mm
- net +5V: track 198.2 -> 196.3 mm
- net Vbat: track 38.7 -> 40.3 mm
- net Net-(R15-Pad2): track 52.5 -> 53.8 mm
- net /RXD: track 99.5 -> 100.7 mm

Commit message: update,
Routing:
- net GND: track 405.3 -> 419.8 mm, vias 54 -> 58
- net /DHT_OUT: track 21.1 -> 27.5 mm
- net /esp-12e/nRST: track 72.9 -> 66.9 mm
- net +5V: track 196.3 -> 200.6 mm
- net /esp-12e/usb_to_uart/DTR: track 23.5 -> 19.5 mm, vias 2 -> 1
- net /sunlight_uv/EN: track 62.0 -> 58.8 mm
- net /esp-12e/GPIO2: track 50.0 -> 53.0 mm
- net /esp-12e/GPIO0: track 62.6 -> 64.9 mm
- net +3V3: track 302.7 -> 300.7 mm
- net /esp-12e/usb_to_uart/RTS: track 13.2 -> 13.7 mm

Commit message: update,
Routing:
- net +3V3: track 300.7 -> 302.4 mm
- net Vbat: track 40.7 -> 40.1 mm

Commit message: update,
Routing:
- net /TXD: track 98.6 -> 100.9 mm
- net GND: track 419.7 -> 421.1 mm

Commit message: update,
Parts:
- moved C11 0.50 mm to (114.4, 64.9)
- moved J10 0.50 mm to (109.5, 68.3)
- moved RN4 0.50 mm to (105.8, 60.7)
- moved RN5 0.50 mm to (105.8, 56.0)
- moved U10 0.50 mm to (94.6, 56.0)
- moved U8 0.50 mm to (114.8, 64.9)
- moved U9 0.50 mm to (94.6, 60.5)
Routing:
- net +3V3: track 302.8 -> 288.3 mm, vias 15 -> 14
- net GND: track 421.1 -> 431.9 mm, vias 58 -> 60
- net Net-(C3-Pad1): track 9.99 -> 19.1 mm, vias 0 -> 2
- net /SCL: track 140.8 -> 135.9 mm
- net +5V: track 200.6 -> 202.8 mm
- net /RXD: track 100.7 -> 102.8 mm
- net /TXD: track 100.9 -> 99.3 mm
- net /sunlight_uv/EN: track 58.8 -> 57.3 mm
- net /esp-12e/usb_to_uart/USB_P: track 14.9 -> 13.9 mm
- net Vbat: track 40.1 -> 40.9 mm
- net /esp-12e/usb_to_uart/USB_N: track 14.3 -> 13.8 mm
