File: hardware/cowin-tryout.kicad_pcb (KiCad board)
At the start: 2 copper layers, 63 x 58 mm, 94 parts, among them J1 BMP180_HEADER, J10 USB_DBG, J2 CONN_PMS, J3 SHT3x_HEADER, J7 DEBUG_HEADER, J8 BAT, J9 DHT22_HEADER, Q1 SS9013_J3, Q2 SS9013_J3, SW1 FLASH_BUTTON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

Commit message: update,
Parts:
- moved U13 3.15 mm to (101.0, 104.8)
- moved U12 1.08 mm to (101.0, 108.5)
- moved U15 0.49 mm to (101.0, 106.8)
Routing:
- net Net-(R15-Pad2): track 53.8 -> 52.3 mm, vias 4 -> 3
Changed lines of the file:
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@@
     (thickness 1.6)
     (drawings 23)
-    (tracks 1244)
+    (tracks 1240)
     (zones 0)
     (modules 94)
@@
   (page A4)
   (layers
-    (0 F.Cu signal hide)
-    (31 B.Cu signal hide)
+    (0 F.Cu signal)
+    (31 B.Cu signal)
     (32 B.Adhes user)
     (33 F.Adhes user)
@@
     (solder_mask_min_width 0.25)
     (aux_axis_origin 0 0)
-    (visible_elements FFFF7F7F)
+    (visible_elements FFFFFF7F)
     (pcbplotparams
       (layerselection 0x010fc_ffffffff)
@@
   )
   (module footprint-lib:BOARD_REVISION (layer F.Cu)
-    (at 100.975 106.3)
+    (at 101 106.79)
     (fp_text reference U15 (at 0 0.5) (layer F.SilkS) hide
       (effects (font (size 1 1) (thickness 0.15)))
@@
       (effects (font (size 1 1) (thickness 0.15)))
     )
-    (fp_text user BOARD_REVISION (at 0 0) (layer B.SilkS)
-      (effects (font (size 1 1) (thickness 0.2)) (justify mirror))
+    (fp_text user REV_20190703_print1 (at 0 0) (layer B.SilkS)
+      (effects (font (size 0.8 0.8) (thickness 0.2)) (justify mirror))
     )
     (fp_text user BOARD_REVISION (at 0 0) (layer F.SilkS) hide
@@
   )
   (module footprint-lib:DESIGNED_IN_HONG_KONG (layer F.Cu)
-    (at 100.975 109.607)
+    (at 100.975 108.532)
     (fp_text reference U12 (at 0 0.5) (layer F.SilkS) hide
       (effects (font (size 1 1) (thickness 0.15)))
@@
     )
     (fp_text user "designed in hong kong" (at 0 0) (layer B.SilkS)
-      (effects (font (size 1 1) (thickness 0.15)) (justify mirror))
+      (effects (font (size 0.8 0.8) (thickness 0.15)) (justify mirror))
     )
     (pad "" connect circle (at 0 -2.032) (size 1.524 1.524) (layers Dwgs.User))
   )
   (module footprint-lib:GITHUB_ADDRESS (layer F.Cu)
-    (at 100.975 107.94)
+    (at 101 104.79)
     (fp_text reference U13 (at 0 0.5) (layer F.SilkS) hide
       (effects (font (size 1 1) (thickness 0.15)))
@@
       (effects (font (size 1 1) (thickness 0.15)))
     )
-    (fp_text user github.com/louiscklaw (at 0 0) (layer B.SilkS)
-      (effects (font (size 1 1) (thickness 0.15)) (justify mirror))
+    (fp_text user github.com/louiscklaw/cowin-tryout (at 0 0) (layer B.SilkS)
+      (effects (font (size 0.8 0.8) (thickness 0.15)) (justify mirror))
     )
     (fp_text user github.com/louiscklaw (at 0 0) (layer F.SilkS) hide
@@
     (tags "CMS SOT")
     (attr smd)
-    (fp_text reference U11 (at 0 -4.5) (layer F.SilkS)
+    (fp_text reference U11 (at 0 0 90) (layer F.SilkS)
       (effects (font (size 1 1) (thickness 0.15)))
     )
@@
     (at 60 77 90)
     (attr smd)
-    (fp_text reference U4 (at -0.583644 -1.91413 90) (layer F.SilkS)
-      (effects (font (size 0.482349 0.482349) (thickness 0.05)))
+    (fp_text reference U4 (at 0 2.25 90) (layer F.SilkS)
+      (effects (font (size 1 1) (thickness 0.15)))
     )
     (fp_text value SHT3x-DIS (at -0.27733 1.90426 90) (layer F.SilkS) hide
@@
     (tags "SPST button tactile switch")
     (attr smd)
-    (fp_text reference SW2 (at 0 -0.2 90) (layer F.SilkS)
+    (fp_text reference SW2 (at -0.32 0.05 90) (layer F.SilkS)
       (effects (font (size 1 1) (thickness 0.15)))
     )
@@
     (tags "resistor handsolder")
     (attr smd)
-    (fp_text reference R1 (at 0.9 1.5) (layer F.SilkS)
+    (fp_text reference R1 (at 1.65 3.25) (layer F.SilkS)
       (effects (font (size 1 1) (thickness 0.15)))
     )
@@
     (descr "Through hole straight pin header, 1x06, 1.27mm pitch, single row")
     (tags "Through hole pin header THT 1x06 1.27mm single row")
-    (fp_text reference J3 (at 0 -1.695) (layer F.SilkS)
+    (fp_text reference J3 (at 0 -2) (layer F.SilkS)
       (effects (font (size 1 1) (thickness 0.15)))
     )
@@
     (tags "capacitor handsolder")
     (attr smd)
-    (fp_text reference C5 (at -0.2 1.5) (layer F.SilkS)
+    (fp_text reference C5 (at -1.45 -3.75) (layer F.SilkS)
       (effects (font (size 1 1) (thickness 0.15)))
     )
@@
     (tags "capacitor handsolder")
     (attr smd)
-    (fp_text reference C3 (at 0 1.15) (layer F.SilkS)
+    (fp_text reference C3 (at -3.45 -4.85) (layer F.SilkS)
       (effects (font (size 1 1) (thickness 0.15)))
     )
@@
     (tags "capacitor handsolder")
     (attr smd)
-    (fp_text reference C2 (at 0 -1.43) (layer F.SilkS)
+    (fp_text reference C2 (at -3.45 -4.55) (layer F.SilkS)
       (effects (font (size 1 1) (thickness 0.15)))
     )
@@
   (segment (start 116.025 64.9) (end 116.038 64.8875) (width 0.5) (layer B.Cu) (net 2))
   (via (at 59.81 95.4211) (size 0.8) (layers F.Cu B.Cu) (net 2))
-  (via (at 116.038 64.8875) (size 0.8) (drill 0.4) (layers F.Cu B.Cu) (net 2) (status 1000000))
+  (via (at 116.038 64.8875) (size 0.8) (drill 0.4) (layers F.Cu B.Cu) (net 2))
   (segment (start 61.835 72.136) (end 69.342 72.136) (width 0.6) (layer F.Cu) (net 2) (status 10))
   (segment (start 70.5375 70.9405) (end 70.5375 69.905) (width 0.6) (layer F.Cu) (net 2) (status 20))
@@
   (segment (start 67.71 90.92) (end 69.715 92.925) (width 0.25) (layer F.Cu) (net 35))
   (segment (start 67.71 89.92) (end 67.71 90.92) (width 0.25) (layer F.Cu) (net 35) (status 10))
-  (segment (start 76.1863 89.8498) (end 75.9455 89.8498) (width 0.25) (layer F.Cu) (net 36))
-  (segment (start 75.9455 89.8498) (end 75.8753 89.92) (width 0.25) (layer F.Cu) (net 36))
-  (segment (start 74.8 89.92) (end 75.8753 89.92) (width 0.25) (layer F.Cu) (net 36) (status 10))
-  (via (at 76.1863 89.8498) (size 0.8) (layers F.Cu B.Cu) (net 36))
   (via (at 91.186 85.09) (size 0.8) (drill 0.4) (layers F.Cu B.Cu) (net 36))
   (via (at 78 94.675) (size 0.8) (drill 0.4) (layers F.Cu B.Cu) (net 36) (status 30))

Commit message: update,
Routing:
- net /esp-12e/ADC: vias 3 -> 2
Changed lines of the file:
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@@
     (thickness 1.6)
     (drawings 23)
-    (tracks 1240)
+    (tracks 1238)
     (zones 0)
     (modules 94)
@@
   (via (at 102.064616 82.126697) (size 0.8) (drill 0.4) (layers F.Cu B.Cu) (net 2))
   (via (at 106.13 96.02) (size 0.6) (drill 0.4) (layers F.Cu B.Cu) (net 2))
-  (via (at 105.06 99.52) (size 0.6) (drill 0.4) (layers F.Cu B.Cu) (net 2))
+  (via (at 104.75 99.75) (size 0.6) (drill 0.4) (layers F.Cu B.Cu) (net 2))
   (via (at 106.19 89.45) (size 0.6) (drill 0.4) (layers F.Cu B.Cu) (net 2))
   (via (at 89.05 58.87) (size 0.6) (drill 0.4) (layers F.Cu B.Cu) (net 2))
@@
   (segment (start 108.7222 87.035021) (end 109.708947 87.035021) (width 0.25) (layer F.Cu) (net 36))
   (segment (start 91.585999 85.489999) (end 107.177178 85.489999) (width 0.25) (layer F.Cu) (net 36))
-  (via (at 104.85 101.35) (size 0.8) (drill 0.4) (layers F.Cu B.Cu) (net 37))
   (segment (start 105.7 100.5) (end 104.85 101.35) (width 0.25) (layer F.Cu) (net 37))
   (segment (start 108.6 100.5) (end 105.7 100.5) (width 0.25) (layer F.Cu) (net 37) (status 10))
@@
   (segment (start 104.815667 98.374333) (end 102.96 100.23) (width 0.25) (layer F.Cu) (net 48))
   (segment (start 104.815667 96.044333) (end 104.815667 98.374333) (width 0.25) (layer F.Cu) (net 48))
-  (segment (start 105.895 100.875) (end 105.25 100.23) (width 0.25) (layer B.Cu) (net 48))
-  (segment (start 112 100.875) (end 105.895 100.875) (width 0.25) (layer B.Cu) (net 48) (status 10))
-  (segment (start 105.25 100.23) (end 102.96 100.23) (width 0.25) (layer B.Cu) (net 48))
   (segment (start 108.6 90.5) (end 107.1 90.5) (width 0.25) (layer F.Cu) (net 48) (status 10))
   (segment (start 106.5105 92.3505) (end 104.815667 94.045333) (width 0.25) (layer F.Cu) (net 48))
@@
   (segment (start 107.1 90.5) (end 106.5105 91.0895) (width 0.25) (layer F.Cu) (net 48))
   (segment (start 106.5105 91.0895) (end 106.5105 92.3505) (width 0.25) (layer F.Cu) (net 48))
+  (segment (start 103.605 100.875) (end 102.96 100.23) (width 0.25) (layer B.Cu) (net 48))
+  (segment (start 112 100.875) (end 103.605 100.875) (width 0.25) (layer B.Cu) (net 48))
   (segment (start 113.3375 64.25) (end 111.6 64.25) (width 0.25) (layer F.Cu) (net 49) (status 10))
   (segment (start 111.6 64.25) (end 110.9 63.55) (width 0.25) (layer F.Cu) (net 49))

Commit message: update,
Routing:
- net GND: vias 60 -> 61
Changed lines of the file:
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@@
     (thickness 1.6)
     (drawings 23)
-    (tracks 1238)
+    (tracks 1240)
     (zones 0)
     (modules 94)
@@
   (segment (start 90.07 64.1) (end 96.7 64.1) (width 0.6) (layer B.Cu) (net 2))
   (via (at 98.45 58.3) (size 0.8) (drill 0.4) (layers F.Cu B.Cu) (net 2))
-  (via (at 101.25 58.3) (size 0.8) (drill 0.4) (layers F.Cu B.Cu) (net 2))
-  (segment (start 94.6 56) (end 94.6 60.5) (width 0.6) (layer B.Cu) (net 2) (status 30))
+  (via (at 101 58.75) (size 0.8) (drill 0.4) (layers F.Cu B.Cu) (net 2))
+  (segment (start 94.6 56) (end 94.6 58.15) (width 0.6) (layer B.Cu) (net 2) (status 30))
   (segment (start 94.6 62) (end 96.7 64.1) (width 0.6) (layer F.Cu) (net 2))
   (segment (start 94.6 60.5) (end 94.6 62) (width 0.6) (layer F.Cu) (net 2) (status 10))
@@
   (segment (start 98.200001 65.949999) (end 97.675 66.475) (width 0.6) (layer F.Cu) (net 2))
   (segment (start 100.600001 65.949999) (end 98.200001 65.949999) (width 0.6) (layer F.Cu) (net 2))
+  (segment (start 94.6 58.15) (end 94.6 60.5) (width 0.6) (layer B.Cu) (net 2) (status 30))
+  (via (at 94.6 58.25) (size 0.8) (drill 0.4) (layers F.Cu B.Cu) (net 2))
   (via (at 62.02 97.67) (size 0.8) (drill 0.4) (layers F.Cu B.Cu) (net 3))
   (segment (start 62.02 97.67) (end 62.02 100.2) (width 0.25) (layer F.Cu) (net 3))

Commit message: update,
Parts:
- J8: footprint Connector_PinHeader_2.54mm:PinHeader_1x02_P2.54mm_Vertical -> kicad-jst-xh.pretty:JST_B2B-XH-A-2.54
- moved J8 2.02 mm to (114.0, 78.7), turned to 90 degrees
- moved J7 1.20 mm to (113.5, 71.3)
- moved Q2 0.59 mm to (113.9, 83.5)
- moved R17 0.58 mm to (111.2, 83.5)
- moved R18 0.54 mm to (111.2, 83.5)
- moved Q1 0.54 mm to (113.9, 83.5)
Routing:
- net GND: track 431.9 -> 436.0 mm
- net Vbat: track 40.9 -> 42.8 mm
- net /esp-12e/GPIO2: track 53.0 -> 54.8 mm
- net +5V: track 202.8 -> 204.3 mm
- net /esp-12e/nRST: track 66.9 -> 68.3 mm
- net /esp-12e/usb_to_uart/DTR: track 19.5 -> 20.7 mm
- net /esp-12e/GPIO0: track 64.9 -> 65.9 mm
- net Net-(R15-Pad2): vias 3 -> 2

Commit message: update,
Routing:
- net /GPIO12: track 69.6 -> 69.0 mm
Other:
- board text added: "+"
Changed lines of the file:
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@@
   (general
     (thickness 1.6)
-    (drawings 23)
-    (tracks 1263)
+    (drawings 24)
+    (tracks 1265)
     (zones 0)
     (modules 94)
@@
     (descr "JST XH series connector, JST_B2B-XH-A")
     (tags "connector jst xh")
-    (fp_text reference J8 (at 2.5 -1.25 180) (layer B.SilkS)
+    (fp_text reference J8 (at 2.5 -1.25) (layer B.SilkS)
       (effects (font (size 1 1) (thickness 0.15)) (justify mirror))
     )
@@
       (effects (font (size 1 1) (thickness 0.15)) (justify mirror))
     )
-    (pad 2 thru_hole circle (at 2.54 0 90) (size 1.5 1.5) (drill 1) (layers *.Cu *.Mask B.SilkS)
+    (pad 2 thru_hole circle (at 2.54 0 90) (size 2 2) (drill 1.4) (layers *.Cu *.Mask B.SilkS)
       (net 41 Vbat))
-    (pad 1 thru_hole rect (at 0 0 90) (size 1.5 1.5) (drill 0.9) (layers *.Cu *.Mask B.SilkS)
+    (pad 1 thru_hole rect (at 0 0 90) (size 2 2) (drill 1.4) (layers *.Cu *.Mask B.SilkS)
       (net 2 GND))
     (model /home/logic/_workspace/kicad/kicad_library/kicad-packages3d/kicad-jst-xh-2.54.3dshapes/JST_B2B-XH-A-2.54.wrl
@@
     (at 113.9 83.5 90)
     (descr SOT23)
-    (fp_text reference Q2 (at -2.8 0.15 90) (layer B.SilkS)
+    (fp_text reference Q2 (at -2.75 0.1 90) (layer B.SilkS)
       (effects (font (size 1 1) (thickness 0.15)) (justify mirror))
     )
@@
     (tags "capacitor handsolder")
     (attr smd)
-    (fp_text reference C14 (at 3.15 -0.85) (layer B.SilkS)
+    (fp_text reference C14 (at -0.85 6.65) (layer B.SilkS)
       (effects (font (size 1 1) (thickness 0.15)) (justify mirror))
     )
@@
     (tags "capacitor handsolder")
     (attr smd)
-    (fp_text reference C13 (at 3.15 -1.65 180) (layer B.SilkS)
+    (fp_text reference C13 (at -0.85 5.85 180) (layer B.SilkS)
       (effects (font (size 1 1) (thickness 0.15)) (justify mirror))
     )
@@
     (tags "capacitor handsolder")
     (attr smd)
-    (fp_text reference C12 (at 3.15 -1.95) (layer B.SilkS)
+    (fp_text reference C12 (at -0.85 5.55) (layer B.SilkS)
       (effects (font (size 1 1) (thickness 0.15)) (justify mirror))
     )
@@
     )
   )
+  (gr_text + (at 110.75 72.25 270) (layer B.SilkS)
+    (effects (font (size 2 2) (thickness 0.3)) (justify mirror))
+  )
   (gr_line (start 118 70) (end 118 108) (layer Edge.Cuts) (width 0.05))
   (gr_line (start 118 60) (end 118 56) (layer Edge.Cuts) (width 0.05))
@@
   (segment (start 75.92 56.6753) (end 75.946 56.7013) (width 0.25) (layer F.Cu) (net 20))
   (segment (start 75.946 56.7013) (end 75.946 58.411) (width 0.25) (layer F.Cu) (net 20) (status 20))
-  (segment (start 110.8897 91.049) (end 110.8897 91.7856) (width 0.25) (layer F.Cu) (net 20))
-  (segment (start 110.8897 91.7856) (end 110.1753 92.5) (width 0.25) (layer F.Cu) (net 20))
-  (segment (start 108.6 92.5) (end 110.1753 92.5) (width 0.25) (layer F.Cu) (net 20) (status 10))
   (segment (start 75.92 55.5) (end 75.92 56.6753) (width 0.25) (layer F.Cu) (net 20) (status 10))
-  (via (at 110.8897 91.049) (size 0.8) (layers F.Cu B.Cu) (net 20))
   (via (at 81.807565 66.471234) (size 0.8) (drill 0.4) (layers F.Cu B.Cu) (net 20))
   (segment (start 81.807565 63.877565) (end 81.807565 66.471234) (width 0.25) (layer B.Cu) (net 20))
@@
   (segment (start 75.92 55.5) (end 75.92 57.99) (width 0.25) (layer B.Cu) (net 20) (status 10))
   (via (at 84.510746 69.740746) (size 0.8) (drill 0.4) (layers F.Cu B.Cu) (net 20))
-  (segment (start 87.040459 67.211033) (end 84.510746 69.740746) (width 0.25) (layer B.Cu) (net 20))
-  (segment (start 104.8384 74.9239) (end 104.8384 72.7737) (width 0.25) (layer B.Cu) (net 20))
-  (segment (start 106.79225 85.619247) (end 106.79225 76.87775) (width 0.25) (layer B.Cu) (net 20))
   (segment (start 84.510746 69.174415) (end 84.510746 69.740746) (width 0.25) (layer F.Cu) (net 20))
-  (segment (start 99.275733 67.211033) (end 87.040459 67.211033) (width 0.25) (layer B.Cu) (net 20))
-  (segment (start 110.8897 89.716697) (end 106.79225 85.619247) (width 0.25) (layer B.Cu) (net 20))
-  (segment (start 106.79225 76.87775) (end 104.8384 74.9239) (width 0.25) (layer B.Cu) (net 20))
-  (segment (start 104.8384 72.7737) (end 99.275733 67.211033) (width 0.25) (layer B.Cu) (net 20))
-  (segment (start 110.8897 91.049) (end 110.8897 89.716697) (width 0.25) (layer B.Cu) (net 20))
   (segment (start 81.807565 66.471234) (end 84.510746 69.174415) (width 0.25) (layer F.Cu) (net 20))
+  (segment (start 110.75 89.576997) (end 110.75 89.934315) (width 0.25) (layer B.Cu) (net 20))
+  (segment (start 110.75 89.934315) (end 110.75 90.5) (width 0.25) (layer B.Cu) (net 20))
+  (segment (start 104.8384 72.7737) (end 104.8384 74.9239) (width 0.25) (layer B.Cu) (net 20))
+  (segment (start 106.79225 85.619247) (end 110.75 89.576997) (width 0.25) (layer B.Cu) (net 20))
+  (segment (start 106.79225 76.87775) (end 106.79225 85.619247) (width 0.25) (layer B.Cu) (net 20))
+  (segment (start 104.8384 74.9239) (end 106.79225 76.87775) (width 0.25) (layer B.Cu) (net 20))
+  (segment (start 87.040459 67.211033) (end 99.275733 67.211033) (width 0.25) (layer B.Cu) (net 20))
+  (segment (start 84.510746 69.740746) (end 87.040459 67.211033) (width 0.25) (layer B.Cu) (net 20))
+  (segment (start 110.75 91.1) (end 110.75 91.065685) (width 0.25) (layer F.Cu) (net 20))
+  (segment (start 110.75 91.065685) (end 110.75 90.5) (width 0.25) (layer F.Cu) (net 20))
+  (segment (start 99.275733 67.211033) (end 104.8384 72.7737) (width 0.25) (layer B.Cu) (net 20))
+  (segment (start 109.35 92.5) (end 110.75 91.1) (width 0.25) (layer F.Cu) (net 20))
+  (segment (start 108.6 92.5) (end 109.35 92.5) (width 0.25) (layer F.Cu) (net 20))
+  (via (at 110.75 90.5) (size 0.8) (drill 0.4) (layers F.Cu B.Cu) (net 20))
   (segment (start 71.15 75.8) (end 72 76.65) (width 0.25) (layer F.Cu) (net 21) (status 20))
   (segment (start 67.05 75.8) (end 71.15 75.8) (width 0.25) (layer F.Cu) (net 21) (status 10))
@@
   (segment (start 102.271899 83.10499) (end 102.271899 89.2681) (width 0.25) (layer B.Cu) (net 23))
   (segment (start 116.04 73.76) (end 116.04 71.3) (width 0.25) (layer F.Cu) (net 23))
-  (segment (start 116.04 79.319978) (end 116.04 73.76) (width 0.25) (layer F.Cu) (net 23))
+  (segment (start 116.04 79.96) (end 116.04 73.76) (width 0.25) (layer F.Cu) (net 23))
   (segment (start 106.20499 83.10499) (end 108.9 85.8) (width 0.25) (layer F.Cu) (net 23))
-  (segment (start 108.9 85.8) (end 112.96359 85.8) (width 0.25) (layer F.Cu) (net 23))
-  (segment (start 113.929989 84.833601) (end 113.929989 81.429989) (width 0.25) (layer F.Cu) (net 23))
   (segment (start 102.271899 83.10499) (end 106.20499 83.10499) (width 0.25) (layer F.Cu) (net 23))
+  (segment (start 108.9 85.8) (end 112.96359 85.8) (width 0.25) (layer F.Cu) (net 23))
+  (segment (start 113.929989 82.070011) (end 116.04 79.96) (width 0.25) (layer F.Cu) (net 23))
   (segment (start 112.96359 85.8) (end 113.929989 84.833601) (width 0.25) (layer F.Cu) (net 23))
-  (segment (start 113.929989 81.429989) (end 116.04 79.319978) (width 0.25) (layer F.Cu) (net 23))
+  (segment (start 113.929989 84.833601) (end 113.929989 82.070011) (width 0.25) (layer F.Cu) (net 23))
   (segment (start 65.35 77.4) (end 65.35 78.2) (width 0.25) (layer F.Cu) (net 24) (status 30))
   (segment (start 59.15 88.9) (end 59.15 87.246252) (width 0.25) (layer F.Cu) (net 24) (status 10))

Commit message: update,
Routing:
- net Vbat: track 42.8 -> 47.2 mm
- net GND: track 436.0 -> 434.8 mm, vias 61 -> 62
Other:
- board text added: "G + D"
