File: hardware/usb_to_uart.sch (KiCad schematic (older format))
At the start: 13 parts, among them Q1 SS9013_J3, Q2 SS9013_J3, U7 CH340T, U8 USB_Micro, Y1 O_12M,3225

Commit message: update,
Changed lines of the file:
@@
 F 0 "U7" H 4875 3093 60  0000 C CNN
 F 1 "CH340T" H 4875 2987 60  0000 C CNN
-F 2 "footprint-lib:CH340T_SSOP-20" H 4875 2881 60  0000 C CNN
+F 2 "footprint-lib:CH340T_SSOP-20" H 4875 2881 60  0001 C CNN
 F 3 "" H 4900 2150 60  0000 C CNN
 	1    4900 2150

Commit message: update,
Connections:
- net +5V: no longer U8.1 (VCC)
- new net VBUS: U8.1 (VCC)
Changed lines of the file:
@@
 EESchema Schematic File Version 4
 LIBS:cowin-tryout-cache
+LIBS:CH340T-tryout-cache
+LIBS:MCP73831-cache
 EELAYER 29 0
 EELAYER END
 $Descr User 8500 5500
 encoding utf-8
-Sheet 11 12
+Sheet 11 13
 Title ""
 Date ""
@@
 	4250 2300 2500 2300
 Wire Wire Line
-	2500 2100 2850 2100
-Wire Wire Line
-	2850 2100 2850 1600
-Wire Wire Line
 	2850 1600 3200 1600
 Connection ~ 3200 1600
@@
 Wire Wire Line
 	2850 1450 2850 1600
-Connection ~ 2850 1600
 $Comp
 L power:+5V #PWR0163
@@
 Text HLabel 6150 4450 0    50   Input ~ 0
 GPIO0
+$Comp
+L power:VBUS #PWR0153
+U 1 1 5D20BE2E
+P 2650 1800
+F 0 "#PWR0153" H 2650 1650 50  0001 C CNN
+F 1 "VBUS" H 2665 1973 50  0000 C CNN
+F 2 "" H 2650 1800 50  0001 C CNN
+F 3 "" H 2650 1800 50  0001 C CNN
+	1    2650 1800
+	1    0    0    -1
+$EndComp
+Wire Wire Line
+	2650 1800 2650 2100
+Wire Wire Line
+	2650 2100 2500 2100
 $EndSCHEMATC

Commit message: update,
Connections:
- net at C16.1, Y1.3: now also U7.9 (XI); no longer U7.10 (XO)
- net at C15.1, Y1.1: now also U7.10 (XO); no longer U7.9 (XI)
Other:
- moved on the sheet: C15, C16
Changed lines of the file:
@@
 F 3 "~" H 3600 2700 50  0001 C CNN
 	1    3600 2700
-	1    0    0    -1
+	-1   0    0    -1
 $EndComp
 Wire Wire Line
@@
 L taobao-c:C22pf,0603 C15
 U 1 1 5D061A62
-P 3400 2900
-F 0 "C15" H 3492 2946 50  0000 L CNN
-F 1 "C22pf,0603" H 3492 2855 50  0000 L CNN
-F 2 "Capacitor_SMD:C_0603_1608Metric_Pad1.05x0.95mm_HandSolder" H 3400 2900 50  0001 C CNN
-F 3 "~" H 3400 2900 50  0001 C CNN
-	1    3400 2900
-	1    0    0    -1
-$EndComp
-$Comp
-L taobao-c:C22pf,0603 C16
-U 1 1 5D06326C
 P 3850 2900
-F 0 "C16" H 3942 2946 50  0000 L CNN
+F 0 "C15" H 3942 2946 50  0000 L CNN
 F 1 "C22pf,0603" H 3942 2855 50  0000 L CNN
 F 2 "Capacitor_SMD:C_0603_1608Metric_Pad1.05x0.95mm_HandSolder" H 3850 2900 50  0001 C CNN
@@
 	1    0    0    -1
 $EndComp
+$Comp
+L taobao-c:C22pf,0603 C16
+U 1 1 5D06326C
+P 3400 2900
+F 0 "C16" H 3309 2946 50  0000 R CNN
+F 1 "C22pf,0603" H 3309 2855 50  0000 R CNN
+F 2 "Capacitor_SMD:C_0603_1608Metric_Pad1.05x0.95mm_HandSolder" H 3400 2900 50  0001 C CNN
+F 3 "~" H 3400 2900 50  0001 C CNN
+	1    3400 2900
+	1    0    0    -1
+$EndComp

Commit message: update,
Parts:
- added J10: USB_DBG, Connector_PinHeader_2.54mm:PinHeader_1x05_P2.54mm_Vertical, symbol Connector:Conn_01x05_Female
Connections:
- net GND: now also J10.5 (Pin_5)
- net VBUS: now also J10.1 (Pin_1)
- net USB_N: now reaches U7.7 (UD-), U8.2 (D-)
- net USB_N: now also J10.2 (Pin_2)
- net USB_P: now reaches U7.6 (UD+), U8.3 (D+)
- net USB_P: now also J10.3 (Pin_3)
- net ID: now reaches U8.4 (ID)
- net ID: now also J10.4 (Pin_4)
- no-connect marks 3 -> 2
Changed lines of the file:
@@
 Wire Wire Line
 	2650 2500 2650 2750
-NoConn ~ 2500 2400
 NoConn ~ 5500 2600
 NoConn ~ 5500 2700
@@
 Wire Wire Line
 	2650 2100 2500 2100
+$Comp
+L Connector:Conn_01x05_Female J10
+U 1 1 5D1B9086
+P 2100 3950
+F 0 "J10" H 1950 4350 50  0000 C CNN
+F 1 "USB_DBG" H 1950 4250 50  0000 C CNN
+F 2 "Connector_PinHeader_2.54mm:PinHeader_1x05_P2.54mm_Vertical" H 2100 3950 50  0001 C CNN
+F 3 "~" H 2100 3950 50  0001 C CNN
+	1    2100 3950
+	-1   0    0    -1
+$EndComp
+$Comp
+L power:VBUS #PWR0195
+U 1 1 5D1BAF94
+P 2700 3550
+F 0 "#PWR0195" H 2700 3400 50  0001 C CNN
+F 1 "VBUS" H 2715 3723 50  0000 C CNN
+F 2 "" H 2700 3550 50  0001 C CNN
+F 3 "" H 2700 3550 50  0001 C CNN
+	1    2700 3550
+	1    0    0    -1
+$EndComp
+Wire Wire Line
+	2700 3550 2700 3750
+Wire Wire Line
+	2700 3750 2300 3750
+Text Label 2900 2200 2    50   ~ 0
+USB_N
+Text Label 2900 2300 2    50   ~ 0
+USB_P
+Text Label 2700 3850 2    50   ~ 0
+USB_N
+Text Label 2700 3950 2    50   ~ 0
+USB_P
+Wire Wire Line
+	2300 3850 2700 3850
+Wire Wire Line
+	2300 3950 2700 3950
+Text Label 2900 2400 2    50   ~ 0
+ID
+Wire Wire Line
+	2900 2400 2500 2400
+Text Label 2700 4050 2    50   ~ 0
+ID
+Wire Wire Line
+	2700 4050 2300 4050
+$Comp
+L power:GND #PWR0196
+U 1 1 5D1C2496
+P 2550 4250
+F 0 "#PWR0196" H 2550 4000 50  0001 C CNN
+F 1 "GND" H 2600 4050 50  0000 C CNN
+F 2 "" H 2550 4250 50  0001 C CNN
+F 3 "" H 2550 4250 50  0001 C CNN
+	1    2550 4250
+	1    0    0    -1
+$EndComp
+Wire Wire Line
+	2550 4250 2550 4150
+Wire Wire Line
+	2550 4150 2300 4150
 $EndSCHEMATC
