File: hardware/pm2_5.sch (KiCad schematic (older format))
At the start: 9 parts

Commit message: update,
Parts:
- D1: renamed from D?; value LED_GREEN -> 5V_HEALTHY
- D2: renamed from D?; value LED_GREEN -> 3V3_HEALTHY
- gave numbers to parts that had none: 7

Commit message: update,
Parts:
- R4, R5: footprint Resistor_SMD:R_0805_2012Metric_Pad1.15x1.40mm_HandSolder -> Resistor_SMD:R_0603_1608Metric_Pad1.05x0.95mm_HandSolder
Changed lines of the file:
@@
 F 0 "R5" H 2300 3250 50  0000 L CNN
 F 1 "R102" H 2300 3200 50  0000 L CNN
-F 2 "Resistor_SMD:R_0805_2012Metric_Pad1.15x1.40mm_HandSolder" H 2200 3200 50  0001 C CNN
+F 2 "Resistor_SMD:R_0603_1608Metric_Pad1.05x0.95mm_HandSolder" H 2200 3200 50  0001 C CNN
 F 3 "~" H 2200 3200 50  0001 C CNN
 	1    2200 3200
@@
 F 0 "R4" H 1650 3250 50  0000 L CNN
 F 1 "R102" H 1650 3200 50  0000 L CNN
-F 2 "Resistor_SMD:R_0805_2012Metric_Pad1.15x1.40mm_HandSolder" H 1550 3200 50  0001 C CNN
+F 2 "Resistor_SMD:R_0603_1608Metric_Pad1.05x0.95mm_HandSolder" H 1550 3200 50  0001 C CNN
 F 3 "~" H 1550 3200 50  0001 C CNN
 	1    1550 3200

Commit message: update,
Parts:
- removed D2: 3V3_HEALTHY, LED_SMD:LED_0805_2012Metric_Pad1.15x1.40mm_HandSolder, symbol taobao-components:LED_GREEN
- removed R5: R102, Resistor_SMD:R_0603_1608Metric_Pad1.05x0.95mm_HandSolder, symbol taobao-r:R102
Changed lines of the file:
@@
 EndData
 $EndBitmap
-$Comp
-L customized_power:+3V3 #PWR0110
-U 1 1 5BC655C0
-P 2200 3000
-F 0 "#PWR0110" H 2200 2850 50  0001 C CNN
-F 1 "+3V3" H 2250 3200 50  0000 C CNN
-F 2 "" H 2200 3000 50  0001 C CNN
-F 3 "" H 2200 3000 50  0001 C CNN
-	1    2200 3000
-	1    0    0    -1
-$EndComp
-Wire Wire Line
-	2200 3000 2200 3100
-Wire Wire Line
-	2200 3300 2200 3400
-Wire Wire Line
-	2200 3600 2200 3700
-$Comp
-L power:GND #PWR0111
-U 1 1 5BC6504F
-P 2200 3700
-F 0 "#PWR0111" H 2200 3450 50  0001 C CNN
-F 1 "GND" H 2250 3500 50  0000 C CNN
-F 2 "" H 2200 3700 50  0001 C CNN
-F 3 "" H 2200 3700 50  0001 C CNN
-	1    2200 3700
-	1    0    0    -1
-$EndComp
-$Comp
-L taobao-components:LED_GREEN D2
-U 1 1 5BC65049
-P 2200 3500
-F 0 "D2" V 2250 3400 50  0000 R CNN
-F 1 "3V3_HEALTHY" V 2200 3400 50  0000 R CNN
-F 2 "LED_SMD:LED_0805_2012Metric_Pad1.15x1.40mm_HandSolder" V 2200 3500 50  0001 C CNN
-F 3 "~" V 2200 3500 50  0001 C CNN
-	1    2200 3500
-	0    -1   -1   0
-$EndComp
-$Comp
-L taobao-r:R102 R5
-U 1 1 5BC65043
-P 2200 3200
-F 0 "R5" H 2300 3250 50  0000 L CNN
-F 1 "R102" H 2300 3200 50  0000 L CNN
-F 2 "Resistor_SMD:R_0603_1608Metric_Pad1.05x0.95mm_HandSolder" H 2200 3200 50  0001 C CNN
-F 3 "~" H 2200 3200 50  0001 C CNN
-	1    2200 3200
-	1    0    0    -1
-$EndComp
 Wire Wire Line
 	1550 3000 1550 3100
