File: hardware/esp-12e.sch (KiCad schematic (older format))
At the start: 13 parts, among them J6 I2C_HEADER,2.54, J7 DEBUG_HEADER, U6 ESP12

Commit message: update,
Connections:
- no-connect marks 11 -> 10
Changed lines of the file:
@@
 $Descr A4 11693 8268
 encoding utf-8
-Sheet 9 14
+Sheet 9 15
 Title ""
 Date ""
@@
 Text Label 1650 6200 0    50   ~ 0
 GPIO12
-Text Label 1650 6300 0    50   ~ 0
-GPIO13
 Text Label 1650 6700 0    50   ~ 0
 SPI_MOSI
@@
 Wire Wire Line
 	3100 1850 2700 1850
-NoConn ~ 1650 6300
 $Comp
 L taobao-r:R471,0603 R12
@@
 Wire Wire Line
 	3600 4100 3600 5350
+Text Label 1650 6300 0    50   ~ 0
+GPIO13
 $EndSCHEMATC

Commit message: update,
Parts:
- added R?: R224,0805, Resistor_SMD:R_0805_2012Metric_Pad1.15x1.40mm_HandSolder, symbol taobao-r:R224,0805
- added R?: R104,0603, Resistor_SMD:R_0603_1608Metric_Pad1.05x0.95mm_HandSolder, symbol taobao-r:R104,0603
Connections:
- net ADC: now also R?.1, R?.2
- net GND: now also R?.2
- new net ADC_EX: R?.1
